Commit message: [hector_quadrotor_urdf] -updated model to use .dae generated by exporting .stl from blender and then exporting to .dae via meshlab.

File: hector_quadrotor/hector_quadrotor_urdf/urdf/generic_camera.urdf.xacro (robot description, xacro)
@@ -23,5 +23,7 @@
             <box size="0.05 0.05 0.05" />
           </geometry>
-          <material name="DarkGrey" />
+	  <material name="Blue">
+      <color rgba="0.0 0.0 0.8 1"/>
+    </material>
         </visual>
         <collision>

File: hector_quadrotor/hector_quadrotor_urdf/urdf/hokuyo_utm30lx.urdf.xacro (robot description, xacro)
@@ -23,5 +23,7 @@
 	    <box size="0.05 0.05 0.05" />
 	  </geometry>
-	  <material name="DarkGrey" />
+	  <material name="Blue">
+      <color rgba="0.0 0.0 0.8 1"/>
+    </material>
 	</visual>
 	<collision>

File: hector_quadrotor/hector_quadrotor_urdf/urdf/quadrotor_base.urdf.xacro (robot description, xacro)
@@ -16,5 +16,7 @@
       <origin xyz="0 0 0" rpy="0 0 0" />
       <geometry>
-        <mesh filename="package://hector_quadrotor_urdf/meshes/quadrotor/quadrotor_base.stl"/>
+	      <!--<mesh filename="package://hector_quadrotor_urdf/meshes/quadrotor/quadrotor_dae_from_stl.dae" scale="0.1 0.1 0.1"/>-->
+              <mesh filename="package://hector_quadrotor_urdf/meshes/quadrotor/quadrotor_base_dae_from_stl.dae"/>
+               <!--<cylinder radius="0.4" length="0.2"/>-->
       </geometry>
       <material name="DarkGrey" >

Commit message: hector_gazebo_plugins/hector_quadrotor_urdf: added sonar plugin, cleaned up urdf models

File: hector_quadrotor/hector_quadrotor_urdf/urdf/generic_camera.urdf.xacro (robot description, xacro)
@@ -5,16 +5,15 @@
   xmlns:xacro="http://ros.org/wiki/xacro"
   >
-    <xacro:macro name="generic_camera" params="name parent *origin ros_topic update_rate min_angle max_angle">
+    <xacro:macro name="generic_camera" params="name parent *origin ros_topic update_rate">
       <joint name="${name}_joint" type="fixed">
-        <axis xyz="0 1 0" />
         <insert_block name="origin" />
         <parent link="${parent}"/>
         <child link="${name}_link"/>
       </joint>
-      <link name="${name}_link" type="laser">
+      <link name="${name}_link">
         <inertial>
           <mass value="0.001" />
           <origin xyz="0 0 0" rpy="0 0 0" />
-          <inertia ixx="0.0001" ixy="0" ixz="0" iyy="0.000001" iyz="0" izz="0.0001" />
+          <inertia ixx="0.0001" ixy="0" ixz="0" iyy="0.0001" iyz="0" izz="0.0001" />
         </inertial>
         <visual>
@@ -30,5 +29,5 @@
           <origin xyz="0 0 0" rpy="0 0 0" />
           <geometry>
-            <box size=".05 .05 .05" />
+            <box size="0.05 0.05 0.05" />
           </geometry>
         </collision>
@@ -41,9 +40,9 @@
         <nearClip>0.01</nearClip>
         <farClip>100</farClip>
-        <updateRate>15.0</updateRate>
+        <updateRate>${update_rate}</updateRate>
         <controller:gazebo_ros_camera name="${name}_camera_controller" plugin="libgazebo_ros_camera.so">
           <alwaysOn>true</alwaysOn>
-          <updateRate>15.0</updateRate>
-          <imageTopicName>finger_tip_cam/image</imageTopicName>
+          <updateRate>${update_rate}</updateRate>
+          <imageTopicName>${ros_topic}</imageTopicName>
           <frameName>${name}_link</frameName>
           <interface:camera name="${name}_camera_iface" />

File: hector_quadrotor/hector_quadrotor_urdf/urdf/hokuyo_utm30lx.urdf.xacro (robot description, xacro)
@@ -5,16 +5,15 @@
   xmlns:xacro="http://ros.org/wiki/xacro"
   >
-    <xacro:macro name="hokuyo_utm30lx" params="name parent *origin ros_topic update_rate min_angle max_angle">
+    <xacro:macro name="hokuyo_utm30lx" params="name parent *origin ros_topic update_rate ray_count min_angle max_angle">
       <joint name="${name}_joint" type="fixed">
-	<axis xyz="0 1 0" />
 	<insert_block name="origin" />
 	<parent link="${parent}"/>
 	<child link="${name}_link"/>
       </joint>
-      <link name="${name}_link" type="laser">
+      <link name="${name}_link">
 	<inertial>
 	  <mass value="0.001" />
 	  <origin xyz="0 0 0" rpy="0 0 0" />
-	  <inertia ixx="0.0001" ixy="0" ixz="0" iyy="0.000001" iyz="0" izz="0.0001" />
+		<inertia ixx="0.0001" ixy="0" ixz="0" iyy="0.0001" iyz="0" izz="0.0001" />
 	</inertial>
 	<visual>
@@ -30,5 +29,5 @@
 	  <origin xyz="0 0 0" rpy="0 0 0" />
 	  <geometry>
-	    <box size=".05 .05 .05" />
+			<box size="0.05 0.05 0.05" />
 	  </geometry>
 	</collision>
@@ -36,9 +35,7 @@
       <gazebo reference="${name}_link">
 	<sensor:ray name="${name}">
-	  <rayCount>640</rayCount>
-	  <rangeCount>640</rangeCount>
-	  <laserCount>1</laserCount>
-	  <origin>0.0 0.0 0.0</origin>
-	  <displayRays>false</displayRays>
+		<rayCount>${ray_count}</rayCount>
+		<rangeCount>${ray_count}</rangeCount>
+		<displayRays>false</displayRays>
 	  <minAngle>${min_angle}</minAngle>
 	  <maxAngle>${max_angle}</maxAngle>

File: hector_quadrotor/hector_quadrotor_urdf/urdf/quadrotor.urdf.xacro (robot description, xacro)
@@ -3,5 +3,6 @@
     xmlns:sensor="http://playerstage.sourceforge.net/gazebo/xmlschema/#sensor"
     xmlns:controller="http://playerstage.sourceforge.net/gazebo/xmlschema/#controller"
-    xmlns:interface="http://playerstage.sourceforge.net/gazebo/xmlschema/#interface">
+    xmlns:interface="http://playerstage.sourceforge.net/gazebo/xmlschema/#interface"
+    xmlns:xacro="http://playerstage.sourceforge.net/gazebo/xmlschema/#interface">
     <!-- Included URDF Files -->
     <include filename="$(find hector_quadrotor_urdf)/urdf/quadrotor_base.urdf.xacro" />

File: hector_quadrotor/hector_quadrotor_urdf/urdf/quadrotor_base.urdf.xacro (robot description, xacro)
@@ -1,99 +1,100 @@
 <?xml version="1.0"?>
-<robot
-xmlns:sensor="http://playerstage.sourceforge.net/gazebo/xmlschema/#sensor"
+<robot xmlns:sensor="http://playerstage.sourceforge.net/gazebo/xmlschema/#sensor"
 xmlns:controller="http://playerstage.sourceforge.net/gazebo/xmlschema/#controller"
-  xmlns:interface="http://playerstage.sourceforge.net/gazebo/xmlschema/#interface">
-    <macro name="quadrotor_base_macro">
-      <link name="base_link">
-  <inertial>
-    <mass value="1.316" />
-    <origin xyz="0 0 0" />
-    <inertia ixx="0.0128" ixy="0.0" ixz="0.0"
-    iyy="0.0128" iyz="0.0"
-      izz="0.0218" />
-    </inertial>
-    <visual>
-      <origin xyz="0 0 0" rpy="0 0 0" />
-      <geometry>
-	      <!--<mesh filename="package://hector_quadrotor_urdf/meshes/quadrotor/quadrotor_dae_from_stl.dae" scale="0.1 0.1 0.1"/>-->
-              <mesh filename="package://hector_quadrotor_urdf/meshes/quadrotor/quadrotor_base_dae_from_stl.dae"/>
-               <!--<cylinder radius="0.4" length="0.2"/>-->
-      </geometry>
-      <material name="DarkGrey" >
-        <color rgba="0.3 0.3 0.3 1"/>
-      </material>
-    </visual>
-    <collision>
-      <origin xyz="0 0 0" rpy="0 0 0" />
-      <geometry>
-        <mesh filename="package://hector_quadrotor_urdf/meshes/quadrotor/quadrotor_base.stl"/>
-      </geometry>
-    </collision>
-  </link>
-  <gazebo reference="base_link">
-    <material>Gazebo/White</material>
-    <turnGravityOff>false</turnGravityOff>
-  </gazebo>
-  <gazebo>
-    <canonicalBody>base_link</canonicalBody>
-    <controller:gazebo_ros_force name="gazebo_ros_force" plugin="libgazebo_ros_force.so">
-      <alwaysOn>true</alwaysOn>
-      <updateRate>0.0</updateRate>
-      <bodyName>base_link</bodyName>
-      <topicName>force</topicName>
-    </controller:gazebo_ros_force>
-    <controller:hector_gazebo_quadrotor_simple_controller name="quadrotor_simple_controller" plugin="libhector_gazebo_quadrotor_simple_controller.so">
-      <alwaysOn>true</alwaysOn>
-      <updateRate>0.0</updateRate>
-      <bodyName>base_link</bodyName>
-      <topicName>cmd_vel</topicName>
-      <rollpitch>
-        <proportionalGain>10.0</proportionalGain>
-        <differentialGain>10.0</differentialGain>
-        <limit>0.5</limit>
-      </rollpitch>
-      <yaw>
-        <proportionalGain>1.0</proportionalGain>
-        <differentialGain>1.0</differentialGain>
-        <limit>1.5</limit>
-      </yaw>
-      <velocity_xy>
-        <proportionalGain>3.0</proportionalGain>
-        <differentialGain>3.0</differentialGain>
-        <limit>2</limit>
-      </velocity_xy>
-      <velocity_z>
-        <proportionalGain>5.0</proportionalGain>
-        <differentialGain>1.0</differentialGain>
-        <limit>2</limit>
-      </velocity_z>
-      <maxForce>30</maxForce>
-    </controller:hector_gazebo_quadrotor_simple_controller>
-    <controller:hector_gazebo_ros_imu name="quadrotor_imu_sim" plugin="libhector_gazebo_ros_imu.so">
-      <alwaysOn>true</alwaysOn>
-      <updateRate>100.0</updateRate>
-      <bodyName>base_link</bodyName>
-      <topicName>imu</topicName>
-      <rpyOffsets>0 0 0</rpyOffsets> <!-- deprecated -->
-      <gaussianNoise>0</gaussianNoise>  <!-- deprecated -->
-      <accelDrift>0.5 0.5 0.5</accelDrift>
-      <accelGaussianNoise>0.1 0.1 0.1</accelGaussianNoise>
-      <rateDrift>0.5 0.5 0.5</rateDrift>
-      <rateGaussianNoise>0.1 0.1 0.1</rateGaussianNoise>
-      <headingDrift>0.05</headingDrift>
-      <headingGaussianNoise>0.01</headingGaussianNoise>
-      <!-- default values:
-        <accelOffset>0 0 0</accelOffset>
-        <accelDrift>0 0 0</accelDrift>
-        <accelDriftFrequency>0.0003 0.0003 0.0003</accelDriftFrequency>
-        <accelGaussianNoise>0 0 0</accelGaussianNoise>
-        <rateOffset>0 0 0</rateOffset>
-        <rateDrift>0 0 0</rateDrift>
-        <rateDriftFrequency>0.0003 0.0003 0.0003</rateDriftFrequency>
-        <rateGaussianNoise>0 0 0</rateGaussianNoise>
-        <headingOffset>0</headingOffset>
-        <headingDrift>0</headingDrift>
-        <headingDriftFrequency>0.0003</headingDriftFrequency>
-        <headingGaussianNoise>0</headingGaussianNoise>
+xmlns:interface="http://playerstage.sourceforge.net/gazebo/xmlschema/#interface"
+xmlns:xacro="http://ros.org/wiki/xacro"
+>
+  <include filename="$(find hector_quadrotor_urdf)/urdf/sonar_sensor.urdf.xacro" />
+  <property name="pi" value="3.1415926535897931" />
+  <xacro:macro name="quadrotor_base_macro">
+    <link name="base_link">
+      <inertial>
+        <mass value="1.316" />
+        <origin xyz="0 0 0" />
+        <inertia ixx="0.0128" ixy="0.0" ixz="0.0" iyy="0.0128" iyz="0.0" izz="0.0218" />
+      </inertial>
+      <visual>
+        <origin xyz="0 0 0" rpy="0 0 0" />
+        <geometry>
+          <!--<mesh filename="package://hector_quadrotor_urdf/meshes/quadrotor/quadrotor_dae_from_stl.dae" scale="0.1 0.1 0.1"/>-->
+                <mesh filename="package://hector_quadrotor_urdf/meshes/quadrotor/quadrotor_base_dae_from_stl.dae"/>
+                 <!--<cylinder radius="0.4" length="0.2"/>-->
+        </geometry>
+        <material name="DarkGrey" >
+          <color rgba="0.3 0.3 0.3 1"/>
+        </material>
+      </visual>
+      <collision>
+        <origin xyz="0 0 0" rpy="0 0 0" />
+        <geometry>
+          <mesh filename="package://hector_quadrotor_urdf/meshes/quadrotor/quadrotor_base.stl"/>
+        </geometry>
+      </collision>
+    </link>
+    <gazebo reference="base_link">
+      <material>Gazebo/White</material>
+      <turnGravityOff>false</turnGravityOff>
+    </gazebo>
+    <gazebo>
+      <canonicalBody>base_link</canonicalBody>
+      <controller:gazebo_ros_force name="gazebo_ros_force" plugin="libgazebo_ros_force.so">
+        <alwaysOn>true</alwaysOn>
+        <updateRate>0.0</updateRate>
+        <bodyName>base_link</bodyName>
+        <topicName>force</topicName>
+      </controller:gazebo_ros_force>
+      <!-- controller:hector_gazebo_quadrotor_simple_controller name="quadrotor_simple_controller" plugin="libhector_gazebo_quadrotor_simple_controller.so">
+        <alwaysOn>true</alwaysOn>
+        <updateRate>0.0</updateRate>
+        <bodyName>base_link</bodyName>
+        <topicName>cmd_vel</topicName>
+        <rollpitch>
+          <proportionalGain>10.0</proportionalGain>
+          <differentialGain>10.0</differentialGain>
+          <limit>0.5</limit>
+        </rollpitch>
+        <yaw>
+          <proportionalGain>1.0</proportionalGain>
+          <differentialGain>1.0</differentialGain>
+          <limit>1.5</limit>
+        </yaw>
+        <velocity_xy>
+          <proportionalGain>3.0</proportionalGain>
+          <differentialGain>3.0</differentialGain>
+          <limit>2</limit>
+        </velocity_xy>
+        <velocity_z>
+          <proportionalGain>5.0</proportionalGain>
+          <differentialGain>1.0</differentialGain>
+          <limit>2</limit>
+        </velocity_z>
+        <maxForce>30</maxForce>
+      </controller:hector_gazebo_quadrotor_simple_controller -->
+      <controller:hector_gazebo_ros_imu name="quadrotor_imu_sim" plugin="libhector_gazebo_ros_imu.so">
+        <alwaysOn>true</alwaysOn>
+        <updateRate>100.0</updateRate>
+        <bodyName>base_link</bodyName>
+        <topicName>imu</topicName>
+        <rpyOffsets>0 0 0</rpyOffsets> <!-- deprecated -->
+        <gaussianNoise>0</gaussianNoise>  <!-- deprecated -->
+        <accelDrift>0.5 0.5 0.5</accelDrift>
+        <accelGaussianNoise>0.1 0.1 0.1</accelGaussianNoise>
+        <rateDrift>0.5 0.5 0.5</rateDrift>
+        <rateGaussianNoise>0.1 0.1 0.1</rateGaussianNoise>
+        <headingDrift>0.05</headingDrift>
+        <headingGaussianNoise>0.01</headingGaussianNoise>
+        <!-- default values:
+          <accelOffset>0 0 0</accelOffset>
+          <accelDrift>0 0 0</accelDrift>
+          <accelDriftFrequency>0.0003 0.0003 0.0003</accelDriftFrequency>
+          <accelGaussianNoise>0 0 0</accelGaussianNoise>
+          <rateOffset>0 0 0</rateOffset>
+          <rateDrift>0 0 0</rateDrift>
+          <rateDriftFrequency>0.0003 0.0003 0.0003</rateDriftFrequency>
+          <rateGaussianNoise>0 0 0</rateGaussianNoise>
+          <headingOffset>0</headingOffset>
+          <headingDrift>0</headingDrift>
+          <headingDriftFrequency>0.0003</headingDriftFrequency>
+          <headingGaussianNoise>0</headingGaussianNoise>
         -->
       </controller:hector_gazebo_ros_imu>
@@ -117,4 +118,8 @@
       </controller:gazebo_ros_p3d>
     </gazebo>
-  </macro>
+    <!-- Sonar height sensor -->
+    <sonar_sensor name="sonar" parent="base_link" ros_topic="sonar_height" update_rate="10" min_range="0.03" max_range="6.0" field_of_view="40" ray_count="10">
+      <origin xyz="0.12 0.0 -0.01" rpy="0 ${90*pi/180} 0"/>
+    </sonar_sensor>
+  </xacro:macro>
 </robot>

File: hector_quadrotor/hector_quadrotor_urdf/urdf/quadrotor_hokuyo_utm30lx.urdf.xacro (robot description, xacro)
@@ -3,6 +3,6 @@
 xmlns:sensor="http://playerstage.sourceforge.net/gazebo/xmlschema/#sensor"
 xmlns:controller="http://playerstage.sourceforge.net/gazebo/xmlschema/#controller"
-  xmlns:interface="http://playerstage.sourceforge.net/gazebo/xmlschema/#interface"
-  xmlns:xacro="http://playerstage.sourceforge.net/gazebo/xmlschema/#interface">
+xmlns:interface="http://playerstage.sourceforge.net/gazebo/xmlschema/#interface"
+xmlns:xacro="http://playerstage.sourceforge.net/gazebo/xmlschema/#interface">
     <!-- Included URDF Files -->
     <include filename="$(find hector_quadrotor_urdf)/urdf/quadrotor_base.urdf.xacro" />
@@ -10,10 +10,10 @@
     <quadrotor_base_macro />
     <include filename="$(find hector_quadrotor_urdf)/urdf/hokuyo_utm30lx.urdf.xacro" />
-    <hokuyo_utm30lx name="laser0" parent="base_link" ros_topic="scan" update_rate="40" min_angle="135" max_angle="-135">
+    <xacro:hokuyo_utm30lx name="laser0" parent="base_link" ros_topic="scan" update_rate="40" ray_count="1081" min_angle="135" max_angle="-135">
       <origin xyz="0.0 0.0 -0.08" rpy="0 0 0"/>
-    </hokuyo_utm30lx>
+    </xacro:hokuyo_utm30lx>
     <include filename="$(find hector_quadrotor_urdf)/urdf/generic_camera.urdf.xacro" />
-    <generic_camera name="front_cam" parent="base_link" ros_topic="scan" update_rate="40" min_angle="135" max_angle="-135">
-      <origin xyz="0.1 0.0 -0.08" rpy="0 0 0"/>
-    </generic_camera>
+    <xacro:generic_camera name="front_cam" parent="base_link" ros_topic="camera/image" update_rate="40">
+      <origin xyz="0.05 0.0 -0.08" rpy="0 0 0"/>
+    </xacro:generic_camera>
   </robot>

Commit message: [hector_quadrotor_urdf] -fix camera mounting so using camera display in rviz works correctly

File: hector_quadrotor/hector_quadrotor_urdf/urdf/generic_camera.urdf.xacro (robot description, xacro)
@@ -5,5 +5,6 @@
   xmlns:xacro="http://ros.org/wiki/xacro"
   >
-    <xacro:macro name="generic_camera" params="name parent *origin ros_topic update_rate">
+    <property name="M_PI" value="3.1415926535897931" />
+    <xacro:macro name="generic_camera" params="name parent *origin ros_topic cam_info_topic update_rate">
       <joint name="${name}_joint" type="fixed">
         <insert_block name="origin" />
@@ -20,5 +21,5 @@
           <origin xyz="0 0 0" rpy="0 0 0" />
           <geometry>
-            <box size="0.05 0.05 0.05" />
+            <box size="0.01 0.01 0.01" />
           </geometry>
 	  <material name="Blue">
@@ -29,8 +30,34 @@
           <origin xyz="0 0 0" rpy="0 0 0" />
           <geometry>
-            <box size="0.05 0.05 0.05" />
+            <box size="0.01 0.01 0.01" />
           </geometry>
         </collision>
       </link>
+    <joint name="${name}_optical_joint" type="fixed">
+      <origin xyz="0 0 0" rpy="${-M_PI/2} 0.0 ${-M_PI/2}" />
+      <parent link="${name}_link" />
+      <child link="${name}_optical_frame"/>
+    </joint>
+    <link name="${name}_optical_frame">
+      <inertial>
+        <mass value="0.01" />
+        <origin xyz="0 0 0" />
+        <inertia ixx="0.001"  ixy="0.0"  ixz="0.0"
+                 iyy="0.001"  iyz="0.0"
+                 izz="0.001" />
+      </inertial>
+      <visual>
+        <origin xyz="0 0 0" rpy="0 0 0"/>
+        <geometry>
+          <box size="0.001 0.001 0.001" />
+        </geometry>
+      </visual>
+      <collision>
+        <origin xyz="0 0 0" rpy="0 0 0"/>
+        <geometry>
+          <box size="0.001 0.001 0.001" />
+        </geometry>
+      </collision>
+    </link>
     <gazebo reference="${name}_link">
       <sensor:camera name="${name}_camera_sensor">
@@ -45,5 +72,6 @@
           <updateRate>${update_rate}</updateRate>
           <imageTopicName>${ros_topic}</imageTopicName>
-          <frameName>${name}_link</frameName>
+          <cameraInfoTopicName>${cam_info_topic}</cameraInfoTopicName>
+          <frameName>${name}_optical_frame</frameName>
           <interface:camera name="${name}_camera_iface" />
         </controller:gazebo_ros_camera>

File: hector_quadrotor/hector_quadrotor_urdf/urdf/quadrotor_hokuyo_utm30lx.urdf.xacro (robot description, xacro)
@@ -14,6 +14,6 @@
     </xacro:hokuyo_utm30lx>
     <include filename="$(find hector_quadrotor_urdf)/urdf/generic_camera.urdf.xacro" />
-    <xacro:generic_camera name="front_cam" parent="base_link" ros_topic="camera/image" update_rate="40">
-      <origin xyz="0.05 0.0 -0.08" rpy="0 0 0"/>
+    <xacro:generic_camera name="front_cam" parent="base_link" ros_topic="camera/image" cam_info_topic="camera/camera_info" update_rate="40">
+      <origin xyz="0.05 0.0 -0.06" rpy="0 0 0"/>
     </xacro:generic_camera>
   </robot>
