Commit message: [hector_quadrotor_urdf] -add camera to hokuyo equipped quadrotor

File: hector_quadrotor/hector_quadrotor_urdf/urdf/quadrotor_hokuyo_utm30lx.urdf.xacro (robot description, xacro)
@@ -13,3 +13,7 @@
       <origin xyz="0.0 0.0 -0.08" rpy="0 0 0"/>
     </hokuyo_utm30lx>
+    <include filename="$(find hector_quadrotor_urdf)/urdf/generic_camera.urdf.xacro" />
+    <generic_camera name="front_cam" parent="base_link" ros_topic="scan" update_rate="40" min_angle="135" max_angle="-135">
+      <origin xyz="0.1 0.0 -0.08" rpy="0 0 0"/>
+    </generic_camera>
   </robot>

Commit message: [hector_quadrotor_urdf] -use hector_sensors_description xacro macro for hokuyo utm-30lx lidar

File: hector_quadrotor/hector_quadrotor_urdf/urdf/quadrotor_hokuyo_utm30lx.urdf.xacro (robot description, xacro)
@@ -5,11 +5,12 @@
 xmlns:interface="http://playerstage.sourceforge.net/gazebo/xmlschema/#interface"
 xmlns:xacro="http://playerstage.sourceforge.net/gazebo/xmlschema/#interface">
+    <property name="M_PI" value="3.1415926535897931" />
     <!-- Included URDF Files -->
     <include filename="$(find hector_quadrotor_urdf)/urdf/quadrotor_base.urdf.xacro" />
     <!-- Instantiate quadrotor_base_macro once (has no parameters atm) -->
     <quadrotor_base_macro />
-    <include filename="$(find hector_quadrotor_urdf)/urdf/hokuyo_utm30lx.urdf.xacro" />
+    <include filename="$(find hector_sensors_description)/urdf/hokuyo_utm30lx.urdf.xacro" />
     <xacro:hokuyo_utm30lx name="laser0" parent="base_link" ros_topic="scan" update_rate="40" ray_count="1081" min_angle="135" max_angle="-135">
-      <origin xyz="0.0 0.0 -0.08" rpy="0 0 0"/>
+      <origin xyz="0.0 0.0 -0.097" rpy="${M_PI} 0 0"/>
     </xacro:hokuyo_utm30lx>
     <include filename="$(find hector_quadrotor_urdf)/urdf/generic_camera.urdf.xacro" />
