Commit message: [hector_quadrotor_urdf] -fix package names in urdf.xacro macro

File: hector_quadrotor/hector_quadrotor_urdf/urdf/quadrotor_base.urdf.xacro (robot description, xacro)
@@ -16,5 +16,5 @@
 	    <origin xyz="0 0 0" rpy="0 0 0" />
 	    <geometry>
-	      <mesh filename="package://quadrotor_urdf/meshes/quadrotor/quadrotor_base.stl"/>
+	      <mesh filename="package://hector_quadrotor_urdf/meshes/quadrotor/quadrotor_base.stl"/>
 	    </geometry>
 	    <material name="DarkGrey" >
@@ -25,5 +25,5 @@
 	    <origin xyz="0 0 0" rpy="0 0 0" />
 	    <geometry>
-	      <mesh filename="package://quadrotor_urdf/meshes/quadrotor/quadrotor_base.stl"/>
+	      <mesh filename="package://hector_quadrotor_urdf/meshes/quadrotor/quadrotor_base.stl"/>
 	    </geometry>
 	  </collision>

Commit message: hector_quadrotor: added package hector_quadrotor_gazebo_plugins with simple controller and baro plugins

File: hector_quadrotor/hector_quadrotor_urdf/urdf/quadrotor_base.urdf.xacro (robot description, xacro)
@@ -3,6 +3,6 @@
 xmlns:sensor="http://playerstage.sourceforge.net/gazebo/xmlschema/#sensor"
 xmlns:controller="http://playerstage.sourceforge.net/gazebo/xmlschema/#controller"
-  xmlns:interface="http://playerstage.sourceforge.net/gazebo/xmlschema/#interface">
-    <macro name="quadrotor_base_macro">
+xmlns:interface="http://playerstage.sourceforge.net/gazebo/xmlschema/#interface">
+  <macro name="quadrotor_base_macro">
       <link name="quadrotor_base">
 	<inertial>
@@ -35,12 +35,39 @@
 	<gazebo>
 	  <canonicalBody>quadrotor_base</canonicalBody>
-	  <controller:gazebo_ros_force name="gazebo_ros_force" plugin="libgazebo_ros_force.so">
-	    <alwaysOn>true</alwaysOn>
-	    <update>1000</update>
-	    <updateRate>1000.0</updateRate>
-	    <bodyName>quadrotor_base</bodyName>
-	    <topicName>force</topicName>
-	  </controller:gazebo_ros_force>
-    <controller:hector_gazebo_ros_imu name="quadro_imu_sim" plugin="libhector_gazebo_ros_imu.so">
+		<!-- <controller:gazebo_ros_force name="gazebo_ros_force" plugin="libgazebo_ros_force.so">
+			<alwaysOn>true</alwaysOn>
+			<updateRate>0.0</updateRate>
+			<bodyName>quadrotor_base</bodyName>
+			<topicName>force</topicName>
+		</controller:gazebo_ros_force> -->
+		<controller:hector_gazebo_quadrotor_simple_controller name="quadrotor_simple_controller" plugin="libhector_gazebo_quadrotor_simple_controller.so">
+			<alwaysOn>true</alwaysOn>
+			<updateRate>0.0</updateRate>
+			<bodyName>quadrotor_base</bodyName>
+			<velocityTopicName>cmd_vel</velocityTopicName>
+			<forceTopicName>force</forceTopicName>
+			<rollpitch>
+				<proportionalGain>10.0</proportionalGain>
+				<differentialGain>10.0</differentialGain>
+				<limit>0.5</limit>
+			</rollpitch>
+			<yaw>
+				<proportionalGain>1.0</proportionalGain>
+				<differentialGain>1.0</differentialGain>
+				<limit>1.5</limit>
+			</yaw>
+			<velocity_xy>
+				<proportionalGain>3.0</proportionalGain>
+				<differentialGain>3.0</differentialGain>
+				<limit>2</limit>
+			</velocity_xy>
+			<velocity_z>
+				<proportionalGain>5.0</proportionalGain>
+				<differentialGain>1.0</differentialGain>
+				<limit>2</limit>
+			</velocity_z>
+			<maxForce>30</maxForce>
+		</controller:hector_gazebo_quadrotor_simple_controller>
+    <controller:hector_gazebo_ros_imu name="quadrotor_imu_sim" plugin="libhector_gazebo_ros_imu.so">
       <alwaysOn>true</alwaysOn>
       <updateRate>100.0</updateRate>
@@ -69,6 +96,16 @@
         <headingGaussianNoise>0</headingGaussianNoise>
       -->
-    </controller:hector_gazebo_ros_imu> -->
-	  <controller:gazebo_ros_p3d name="quadro_groundtruth_sim" plugin="libgazebo_ros_p3d.so">
+    </controller:hector_gazebo_ros_imu>
+    <controller:hector_gazebo_ros_baro name="quadrotor_baro_sim" plugin="libhector_gazebo_ros_baro.so">
+      <alwaysOn>true</alwaysOn>
+      <updateRate>10.0</updateRate>
+      <bodyName>quadrotor_base</bodyName>
+      <topicName>pressure_height</topicName>
+      <offset>0</offset>
+      <drift>0.1</drift>
+      <driftFrequency>0.0003</driftFrequency>
+      <gaussianNoise>0.1</gaussianNoise>
+    </controller:hector_gazebo_ros_baro>
+		<controller:gazebo_ros_p3d name="quadrotor_groundtruth_sim" plugin="libgazebo_ros_p3d.so">
 	    <alwaysOn>true</alwaysOn>
 	    <updateRate>100.0</updateRate>
@@ -79,4 +116,4 @@
 	  </controller:gazebo_ros_p3d>
 	</gazebo>
-      </macro>
-    </robot>
+	</macro>
+</robot>

Commit message: [hector_quadrotor_urdf] -change body fixed main coord frame name to base_link for standardization

File: hector_quadrotor/hector_quadrotor_urdf/urdf/quadrotor_base.urdf.xacro (robot description, xacro)
@@ -3,7 +3,7 @@
 xmlns:sensor="http://playerstage.sourceforge.net/gazebo/xmlschema/#sensor"
 xmlns:controller="http://playerstage.sourceforge.net/gazebo/xmlschema/#controller"
-xmlns:interface="http://playerstage.sourceforge.net/gazebo/xmlschema/#interface">
-  <macro name="quadrotor_base_macro">
-      <link name="quadrotor_base">
+  xmlns:interface="http://playerstage.sourceforge.net/gazebo/xmlschema/#interface">
+    <macro name="quadrotor_base_macro">
+      <link name="base_link">
 	<inertial>
 	  <mass value="1.316" />
@@ -29,91 +29,93 @@
 	  </collision>
 	</link>
-	<gazebo reference="quadrotor_base">
-	  <material>Gazebo/Red</material>
+	<gazebo reference="base_link">
+	  <material>Gazebo/White</material>
 	  <turnGravityOff>false</turnGravityOff>
 	</gazebo>
 	<gazebo>
-	  <canonicalBody>quadrotor_base</canonicalBody>
-		<!-- <controller:gazebo_ros_force name="gazebo_ros_force" plugin="libgazebo_ros_force.so">
-			<alwaysOn>true</alwaysOn>
-			<updateRate>0.0</updateRate>
-			<bodyName>quadrotor_base</bodyName>
-			<topicName>force</topicName>
-		</controller:gazebo_ros_force> -->
-		<controller:hector_gazebo_quadrotor_simple_controller name="quadrotor_simple_controller" plugin="libhector_gazebo_quadrotor_simple_controller.so">
-			<alwaysOn>true</alwaysOn>
-			<updateRate>0.0</updateRate>
-			<bodyName>quadrotor_base</bodyName>
-			<velocityTopicName>cmd_vel</velocityTopicName>
-			<forceTopicName>force</forceTopicName>
-			<rollpitch>
-				<proportionalGain>10.0</proportionalGain>
-				<differentialGain>10.0</differentialGain>
-				<limit>0.5</limit>
-			</rollpitch>
-			<yaw>
-				<proportionalGain>1.0</proportionalGain>
-				<differentialGain>1.0</differentialGain>
-				<limit>1.5</limit>
-			</yaw>
-			<velocity_xy>
-				<proportionalGain>3.0</proportionalGain>
-				<differentialGain>3.0</differentialGain>
-				<limit>2</limit>
-			</velocity_xy>
-			<velocity_z>
-				<proportionalGain>5.0</proportionalGain>
-				<differentialGain>1.0</differentialGain>
-				<limit>2</limit>
-			</velocity_z>
-			<maxForce>30</maxForce>
-		</controller:hector_gazebo_quadrotor_simple_controller>
-    <controller:hector_gazebo_ros_imu name="quadrotor_imu_sim" plugin="libhector_gazebo_ros_imu.so">
-      <alwaysOn>true</alwaysOn>
-      <updateRate>100.0</updateRate>
-      <bodyName>quadrotor_base</bodyName>
-      <topicName>imu</topicName>
-      <rpyOffsets>0 0 0</rpyOffsets> <!-- deprecated -->
-      <gaussianNoise>0</gaussianNoise> <!-- deprecated -->
-      <accelDrift>0.5 0.5 0.5</accelDrift>
-      <accelGaussianNoise>0.1 0.1 0.1</accelGaussianNoise>
-      <rateDrift>0.5 0.5 0.5</rateDrift>
-      <rateGaussianNoise>0.1 0.1 0.1</rateGaussianNoise>
-      <headingDrift>0.05</headingDrift>
-      <headingGaussianNoise>0.01</headingGaussianNoise>
-      <!-- default values:
-        <accelOffset>0 0 0</accelOffset>
-        <accelDrift>0 0 0</accelDrift>
-        <accelDriftFrequency>0.0003 0.0003 0.0003</accelDriftFrequency>
-        <accelGaussianNoise>0 0 0</accelGaussianNoise>
-        <rateOffset>0 0 0</rateOffset>
-        <rateDrift>0 0 0</rateDrift>
-        <rateDriftFrequency>0.0003 0.0003 0.0003</rateDriftFrequency>
-        <rateGaussianNoise>0 0 0</rateGaussianNoise>
-        <headingOffset>0</headingOffset>
-        <headingDrift>0</headingDrift>
-        <headingDriftFrequency>0.0003</headingDriftFrequency>
-        <headingGaussianNoise>0</headingGaussianNoise>
-      -->
-    </controller:hector_gazebo_ros_imu>
-    <controller:hector_gazebo_ros_baro name="quadrotor_baro_sim" plugin="libhector_gazebo_ros_baro.so">
-      <alwaysOn>true</alwaysOn>
-      <updateRate>10.0</updateRate>
-      <bodyName>quadrotor_base</bodyName>
-      <topicName>pressure_height</topicName>
-      <offset>0</offset>
-      <drift>0.1</drift>
-      <driftFrequency>0.0003</driftFrequency>
-      <gaussianNoise>0.1</gaussianNoise>
-    </controller:hector_gazebo_ros_baro>
-		<controller:gazebo_ros_p3d name="quadrotor_groundtruth_sim" plugin="libgazebo_ros_p3d.so">
+	  <canonicalBody>base_link</canonicalBody>
+	  <!-- <controller:gazebo_ros_force name="gazebo_ros_force" plugin="libgazebo_ros_force.so">
+	  <alwaysOn>true</alwaysOn>
+	  <updateRate>0.0</updateRate>
+	  <bodyName>quadrotor_base</bodyName>
+	  <topicName>force</topicName>
+	</controller:gazebo_ros_force> -->
+	  <controller:hector_gazebo_quadrotor_simple_controller name="quadrotor_simple_controller" plugin="libhector_gazebo_quadrotor_simple_controller.so">
+	    <alwaysOn>true</alwaysOn>
+	    <updateRate>0.0</updateRate>
+	    <bodyName>base_link</bodyName>
+	    <velocityTopicName>cmd_vel</velocityTopicName>
+	    <forceTopicName>force</forceTopicName>
+	    <rollpitch>
+	      <proportionalGain>10.0</proportionalGain>
+	      <differentialGain>10.0</differentialGain>
+	      <limit>0.5</limit>
+	    </rollpitch>
+	    <yaw>
+	      <proportionalGain>1.0</proportionalGain>
+	      <differentialGain>1.0</differentialGain>
+	      <limit>1.5</limit>
+	    </yaw>
+	    <velocity_xy>
+	      <proportionalGain>3.0</proportionalGain>
+	      <differentialGain>3.0</differentialGain>
+	      <limit>2</limit>
+	    </velocity_xy>
+	    <velocity_z>
+	      <proportionalGain>5.0</proportionalGain>
+	      <differentialGain>1.0</differentialGain>
+	      <limit>2</limit>
+	    </velocity_z>
+	    <maxForce>30</maxForce>
+	  </controller:hector_gazebo_quadrotor_simple_controller>
+	  <controller:hector_gazebo_ros_imu name="quadrotor_imu_sim" plugin="libhector_gazebo_ros_imu.so">
 	    <alwaysOn>true</alwaysOn>
 	    <updateRate>100.0</updateRate>
-	    <bodyName>quadrotor_base</bodyName>
-			<topicName>state</topicName>
-	    <gaussianNoise>0.0</gaussianNoise>
-	    <frameName>map</frameName>
-	  </controller:gazebo_ros_p3d>
-	</gazebo>
+	    <bodyName>base_link</bodyName>
+	    <topicName>imu</topicName>
+	    <rpyOffsets>0 0 0</rpyOffsets>
+	    <!-- deprecated -->
+	    <gaussianNoise>0</gaussianNoise>
+	    <!-- deprecated -->
+	    <accelDrift>0.5 0.5 0.5</accelDrift>
+	    <accelGaussianNoise>0.1 0.1 0.1</accelGaussianNoise>
+	    <rateDrift>0.5 0.5 0.5</rateDrift>
+	    <rateGaussianNoise>0.1 0.1 0.1</rateGaussianNoise>
+	    <headingDrift>0.05</headingDrift>
+	    <headingGaussianNoise>0.01</headingGaussianNoise>
+	    <!-- default values:
+	      <accelOffset>0 0 0</accelOffset>
+	      <accelDrift>0 0 0</accelDrift>
+	      <accelDriftFrequency>0.0003 0.0003 0.0003</accelDriftFrequency>
+	      <accelGaussianNoise>0 0 0</accelGaussianNoise>
+	      <rateOffset>0 0 0</rateOffset>
+	      <rateDrift>0 0 0</rateDrift>
+	      <rateDriftFrequency>0.0003 0.0003 0.0003</rateDriftFrequency>
+	      <rateGaussianNoise>0 0 0</rateGaussianNoise>
+	      <headingOffset>0</headingOffset>
+	      <headingDrift>0</headingDrift>
+	      <headingDriftFrequency>0.0003</headingDriftFrequency>
+	      <headingGaussianNoise>0</headingGaussianNoise>
+	      -->
+	    </controller:hector_gazebo_ros_imu>
+	    <controller:hector_gazebo_ros_baro name="quadrotor_baro_sim" plugin="libhector_gazebo_ros_baro.so">
+	      <alwaysOn>true</alwaysOn>
+	      <updateRate>10.0</updateRate>
+	      <bodyName>base_link</bodyName>
+	      <topicName>pressure_height</topicName>
+	      <offset>0</offset>
+	      <drift>0.1</drift>
+	      <driftFrequency>0.0003</driftFrequency>
+	      <gaussianNoise>0.1</gaussianNoise>
+	    </controller:hector_gazebo_ros_baro>
+	    <controller:gazebo_ros_p3d name="quadrotor_groundtruth_sim" plugin="libgazebo_ros_p3d.so">
+	      <alwaysOn>true</alwaysOn>
+	      <updateRate>100.0</updateRate>
+	      <bodyName>base_link</bodyName>
+	      <topicName>state</topicName>
+	      <gaussianNoise>0.0</gaussianNoise>
+	      <frameName>map</frameName>
+	    </controller:gazebo_ros_p3d>
+	  </gazebo>
 	</macro>
 </robot>

Commit message: hector_quadrotor_gazebo_plugins/quadrotor_simple_controller: z force cannot be negative, removed force subscriber within quadrotor_simple_controller (can be run together with gazebo_ros_force plugin)

File: hector_quadrotor/hector_quadrotor_urdf/urdf/quadrotor_base.urdf.xacro (robot description, xacro)
@@ -6,116 +6,113 @@
     <macro name="quadrotor_base_macro">
       <link name="base_link">
-	<inertial>
-	  <mass value="1.316" />
-	  <origin xyz="0 0 0" />
-	  <inertia ixx="0.0128" ixy="0.0" ixz="0.0"
-	  iyy="0.0128" iyz="0.0"
-	    izz="0.0218" />
-	  </inertial>
-	  <visual>
-	    <origin xyz="0 0 0" rpy="0 0 0" />
-	    <geometry>
-	      <mesh filename="package://hector_quadrotor_urdf/meshes/quadrotor/quadrotor_base.stl"/>
-	    </geometry>
-	    <material name="DarkGrey" >
-	      <color rgba="0.3 0.3 0.3 1"/>
-	    </material>
-	  </visual>
-	  <collision>
-	    <origin xyz="0 0 0" rpy="0 0 0" />
-	    <geometry>
-	      <mesh filename="package://hector_quadrotor_urdf/meshes/quadrotor/quadrotor_base.stl"/>
-	    </geometry>
-	  </collision>
-	</link>
-	<gazebo reference="base_link">
-	  <material>Gazebo/White</material>
-	  <turnGravityOff>false</turnGravityOff>
-	</gazebo>
-	<gazebo>
-	  <canonicalBody>base_link</canonicalBody>
-	  <!-- <controller:gazebo_ros_force name="gazebo_ros_force" plugin="libgazebo_ros_force.so">
-	  <alwaysOn>true</alwaysOn>
-	  <updateRate>0.0</updateRate>
-	  <bodyName>quadrotor_base</bodyName>
-	  <topicName>force</topicName>
-	</controller:gazebo_ros_force> -->
-	  <controller:hector_gazebo_quadrotor_simple_controller name="quadrotor_simple_controller" plugin="libhector_gazebo_quadrotor_simple_controller.so">
-	    <alwaysOn>true</alwaysOn>
-	    <updateRate>0.0</updateRate>
-	    <bodyName>base_link</bodyName>
-	    <velocityTopicName>cmd_vel</velocityTopicName>
-	    <forceTopicName>force</forceTopicName>
-	    <rollpitch>
-	      <proportionalGain>10.0</proportionalGain>
-	      <differentialGain>10.0</differentialGain>
-	      <limit>0.5</limit>
-	    </rollpitch>
-	    <yaw>
-	      <proportionalGain>1.0</proportionalGain>
-	      <differentialGain>1.0</differentialGain>
-	      <limit>1.5</limit>
-	    </yaw>
-	    <velocity_xy>
-	      <proportionalGain>3.0</proportionalGain>
-	      <differentialGain>3.0</differentialGain>
-	      <limit>2</limit>
-	    </velocity_xy>
-	    <velocity_z>
-	      <proportionalGain>5.0</proportionalGain>
-	      <differentialGain>1.0</differentialGain>
-	      <limit>2</limit>
-	    </velocity_z>
-	    <maxForce>30</maxForce>
-	  </controller:hector_gazebo_quadrotor_simple_controller>
-	  <controller:hector_gazebo_ros_imu name="quadrotor_imu_sim" plugin="libhector_gazebo_ros_imu.so">
-	    <alwaysOn>true</alwaysOn>
-	    <updateRate>100.0</updateRate>
-	    <bodyName>base_link</bodyName>
-	    <topicName>imu</topicName>
-	    <rpyOffsets>0 0 0</rpyOffsets>
-	    <!-- deprecated -->
-	    <gaussianNoise>0</gaussianNoise>
-	    <!-- deprecated -->
-	    <accelDrift>0.5 0.5 0.5</accelDrift>
-	    <accelGaussianNoise>0.1 0.1 0.1</accelGaussianNoise>
-	    <rateDrift>0.5 0.5 0.5</rateDrift>
-	    <rateGaussianNoise>0.1 0.1 0.1</rateGaussianNoise>
-	    <headingDrift>0.05</headingDrift>
-	    <headingGaussianNoise>0.01</headingGaussianNoise>
-	    <!-- default values:
-	      <accelOffset>0 0 0</accelOffset>
-	      <accelDrift>0 0 0</accelDrift>
-	      <accelDriftFrequency>0.0003 0.0003 0.0003</accelDriftFrequency>
-	      <accelGaussianNoise>0 0 0</accelGaussianNoise>
-	      <rateOffset>0 0 0</rateOffset>
-	      <rateDrift>0 0 0</rateDrift>
-	      <rateDriftFrequency>0.0003 0.0003 0.0003</rateDriftFrequency>
-	      <rateGaussianNoise>0 0 0</rateGaussianNoise>
-	      <headingOffset>0</headingOffset>
-	      <headingDrift>0</headingDrift>
-	      <headingDriftFrequency>0.0003</headingDriftFrequency>
-	      <headingGaussianNoise>0</headingGaussianNoise>
-	      -->
-	    </controller:hector_gazebo_ros_imu>
-	    <controller:hector_gazebo_ros_baro name="quadrotor_baro_sim" plugin="libhector_gazebo_ros_baro.so">
-	      <alwaysOn>true</alwaysOn>
-	      <updateRate>10.0</updateRate>
-	      <bodyName>base_link</bodyName>
-	      <topicName>pressure_height</topicName>
-	      <offset>0</offset>
-	      <drift>0.1</drift>
-	      <driftFrequency>0.0003</driftFrequency>
-	      <gaussianNoise>0.1</gaussianNoise>
-	    </controller:hector_gazebo_ros_baro>
-	    <controller:gazebo_ros_p3d name="quadrotor_groundtruth_sim" plugin="libgazebo_ros_p3d.so">
-	      <alwaysOn>true</alwaysOn>
-	      <updateRate>100.0</updateRate>
-	      <bodyName>base_link</bodyName>
-	      <topicName>state</topicName>
-	      <gaussianNoise>0.0</gaussianNoise>
-	      <frameName>map</frameName>
-	    </controller:gazebo_ros_p3d>
-	  </gazebo>
-	</macro>
+  <inertial>
+    <mass value="1.316" />
+    <origin xyz="0 0 0" />
+    <inertia ixx="0.0128" ixy="0.0" ixz="0.0"
+    iyy="0.0128" iyz="0.0"
+      izz="0.0218" />
+    </inertial>
+    <visual>
+      <origin xyz="0 0 0" rpy="0 0 0" />
+      <geometry>
+        <mesh filename="package://hector_quadrotor_urdf/meshes/quadrotor/quadrotor_base.stl"/>
+      </geometry>
+      <material name="DarkGrey" >
+        <color rgba="0.3 0.3 0.3 1"/>
+      </material>
+    </visual>
+    <collision>
+      <origin xyz="0 0 0" rpy="0 0 0" />
+      <geometry>
+        <mesh filename="package://hector_quadrotor_urdf/meshes/quadrotor/quadrotor_base.stl"/>
+      </geometry>
+    </collision>
+  </link>
+  <gazebo reference="base_link">
+    <material>Gazebo/White</material>
+    <turnGravityOff>false</turnGravityOff>
+  </gazebo>
+  <gazebo>
+    <canonicalBody>base_link</canonicalBody>
+    <controller:gazebo_ros_force name="gazebo_ros_force" plugin="libgazebo_ros_force.so">
+      <alwaysOn>true</alwaysOn>
+      <updateRate>0.0</updateRate>
+      <bodyName>base_link</bodyName>
+      <topicName>force</topicName>
+    </controller:gazebo_ros_force>
+    <controller:hector_gazebo_quadrotor_simple_controller name="quadrotor_simple_controller" plugin="libhector_gazebo_quadrotor_simple_controller.so">
+      <alwaysOn>true</alwaysOn>
+      <updateRate>0.0</updateRate>
+      <bodyName>base_link</bodyName>
+      <topicName>cmd_vel</topicName>
+      <rollpitch>
+        <proportionalGain>10.0</proportionalGain>
+        <differentialGain>10.0</differentialGain>
+        <limit>0.5</limit>
+      </rollpitch>
+      <yaw>
+        <proportionalGain>1.0</proportionalGain>
+        <differentialGain>1.0</differentialGain>
+        <limit>1.5</limit>
+      </yaw>
+      <velocity_xy>
+        <proportionalGain>3.0</proportionalGain>
+        <differentialGain>3.0</differentialGain>
+        <limit>2</limit>
+      </velocity_xy>
+      <velocity_z>
+        <proportionalGain>5.0</proportionalGain>
+        <differentialGain>1.0</differentialGain>
+        <limit>2</limit>
+      </velocity_z>
+      <maxForce>30</maxForce>
+    </controller:hector_gazebo_quadrotor_simple_controller>
+    <controller:hector_gazebo_ros_imu name="quadrotor_imu_sim" plugin="libhector_gazebo_ros_imu.so">
+      <alwaysOn>true</alwaysOn>
+      <updateRate>100.0</updateRate>
+      <bodyName>base_link</bodyName>
+      <topicName>imu</topicName>
+      <rpyOffsets>0 0 0</rpyOffsets> <!-- deprecated -->
+      <gaussianNoise>0</gaussianNoise>  <!-- deprecated -->
+      <accelDrift>0.5 0.5 0.5</accelDrift>
+      <accelGaussianNoise>0.1 0.1 0.1</accelGaussianNoise>
+      <rateDrift>0.5 0.5 0.5</rateDrift>
+      <rateGaussianNoise>0.1 0.1 0.1</rateGaussianNoise>
+      <headingDrift>0.05</headingDrift>
+      <headingGaussianNoise>0.01</headingGaussianNoise>
+      <!-- default values:
+        <accelOffset>0 0 0</accelOffset>
+        <accelDrift>0 0 0</accelDrift>
+        <accelDriftFrequency>0.0003 0.0003 0.0003</accelDriftFrequency>
+        <accelGaussianNoise>0 0 0</accelGaussianNoise>
+        <rateOffset>0 0 0</rateOffset>
+        <rateDrift>0 0 0</rateDrift>
+        <rateDriftFrequency>0.0003 0.0003 0.0003</rateDriftFrequency>
+        <rateGaussianNoise>0 0 0</rateGaussianNoise>
+        <headingOffset>0</headingOffset>
+        <headingDrift>0</headingDrift>
+        <headingDriftFrequency>0.0003</headingDriftFrequency>
+        <headingGaussianNoise>0</headingGaussianNoise>
+        -->
+      </controller:hector_gazebo_ros_imu>
+      <controller:hector_gazebo_ros_baro name="quadrotor_baro_sim" plugin="libhector_gazebo_ros_baro.so">
+        <alwaysOn>true</alwaysOn>
+        <updateRate>10.0</updateRate>
+        <bodyName>base_link</bodyName>
+        <topicName>pressure_height</topicName>
+        <offset>0</offset>
+        <drift>0.1</drift>
+        <driftFrequency>0.0003</driftFrequency>
+        <gaussianNoise>0.1</gaussianNoise>
+      </controller:hector_gazebo_ros_baro>
+      <controller:gazebo_ros_p3d name="quadrotor_groundtruth_sim" plugin="libgazebo_ros_p3d.so">
+        <alwaysOn>true</alwaysOn>
+        <updateRate>100.0</updateRate>
+        <bodyName>base_link</bodyName>
+        <topicName>state</topicName>
+        <gaussianNoise>0.0</gaussianNoise>
+        <frameName>map</frameName>
+      </controller:gazebo_ros_p3d>
+    </gazebo>
+  </macro>
 </robot>

Commit message: [hector_quadrotor_urdf] -fix mesh filename for quadrotor model

File: hector_quadrotor/hector_quadrotor_urdf/urdf/quadrotor_base.urdf.xacro (robot description, xacro)
@@ -18,5 +18,5 @@
         <geometry>
           <!--<mesh filename="package://hector_quadrotor_urdf/meshes/quadrotor/quadrotor_dae_from_stl.dae" scale="0.1 0.1 0.1"/>-->
-                <mesh filename="package://hector_quadrotor_urdf/meshes/quadrotor/quadrotor_base_dae_from_stl.dae"/>
+                <mesh filename="package://hector_quadrotor_urdf/meshes/quadrotor/quadrotor_base.dae"/>
                  <!--<cylinder radius="0.4" length="0.2"/>-->
         </geometry>
@@ -28,10 +28,10 @@
         <origin xyz="0 0 0" rpy="0 0 0" />
         <geometry>
-          <mesh filename="package://hector_quadrotor_urdf/meshes/quadrotor/quadrotor_base.stl"/>
+          <mesh filename="package://hector_quadrotor_urdf/meshes/quadrotor/quadrotor_base.dae"/>
         </geometry>
       </collision>
     </link>
     <gazebo reference="base_link">
-      <material>Gazebo/White</material>
+<!--      <material>Gazebo/White</material>-->
       <turnGravityOff>false</turnGravityOff>
     </gazebo>
