Commit message: [hector_quadrotor_urdf] -remove obsolete tags from base xacro file

File: hector_quadrotor/hector_quadrotor_urdf/urdf/quadrotor_base.urdf.xacro (robot description, xacro)
@@ -17,11 +17,6 @@
         <origin xyz="0 0 0" rpy="0 0 0" />
         <geometry>
-          <!--<mesh filename="package://hector_quadrotor_urdf/meshes/quadrotor/quadrotor_dae_from_stl.dae" scale="0.1 0.1 0.1"/>-->
                 <mesh filename="package://hector_quadrotor_urdf/meshes/quadrotor/quadrotor_base.dae"/>
-                 <!--<cylinder radius="0.4" length="0.2"/>-->
         </geometry>
-        <material name="DarkGrey" >
-          <color rgba="0.3 0.3 0.3 1"/>
-        </material>
       </visual>
       <collision>
@@ -33,5 +28,4 @@
     </link>
     <gazebo reference="base_link">
-<!--      <material>Gazebo/White</material>-->
       <turnGravityOff>false</turnGravityOff>
     </gazebo>

Commit message: hector_quadrotor/hector_gazebo: added GPS and Magnetometer plugins

File: hector_quadrotor/hector_quadrotor_urdf/urdf/quadrotor_base.urdf.xacro (robot description, xacro)
@@ -103,4 +103,24 @@
         <gaussianNoise>0.1</gaussianNoise>
       </controller:hector_gazebo_ros_baro>
+      <controller:hector_gazebo_ros_magnetic name="quadrotor_magnetic_sim" plugin="libhector_gazebo_ros_magnetic.so">
+        <alwaysOn>true</alwaysOn>
+        <updateRate>10.0</updateRate>
+        <bodyName>base_link</bodyName>
+        <topicName>magnetic</topicName>
+        <offset>0 0 0</offset>
+        <drift>0.1 0.1 0.1</drift>
+        <driftFrequency>0.0003 0.0003 0.0003</driftFrequency>
+        <gaussianNoise>0.1 0.1 0.1</gaussianNoise>
+      </controller:hector_gazebo_ros_magnetic>
+      <controller:hector_gazebo_ros_gps name="quadrotor_gps_sim" plugin="libhector_gazebo_ros_gps.so">
+        <alwaysOn>true</alwaysOn>
+        <updateRate>4.0</updateRate>
+        <bodyName>base_link</bodyName>
+        <topicName>fix</topicName>
+        <velocityTopicName>gps_velocity</velocityTopicName>
+        <velocityDrift>0.1 0.1 0.5</velocityDrift>
+        <gaussianNoise>0.1 0.1 0.1</gaussianNoise>
+        <velocityGaussianNoise>0.1 0.1 0.1</velocityGaussianNoise>
+      </controller:hector_gazebo_ros_gps>
       <controller:gazebo_ros_p3d name="quadrotor_groundtruth_sim" plugin="libgazebo_ros_p3d.so">
         <alwaysOn>true</alwaysOn>
@@ -113,6 +133,6 @@
     </gazebo>
     <!-- Sonar height sensor -->
-    <sonar_sensor name="sonar" parent="base_link" ros_topic="sonar_height" update_rate="10" min_range="0.03" max_range="6.0" field_of_view="40" ray_count="10">
-      <origin xyz="0.12 0.0 -0.01" rpy="0 ${90*pi/180} 0"/>
+    <sonar_sensor name="sonar" parent="base_link" ros_topic="sonar_height" update_rate="10" min_range="0.03" max_range="3.0" field_of_view="40" ray_count="3">
+      <origin xyz="0.12 0.0 -0.02" rpy="0 ${90*pi/180} 0"/>
     </sonar_sensor>
   </xacro:macro>

Commit message: [hector_quadrotor_urdf] -use sonar_sensor now located in hector_sensors_description

File: hector_quadrotor/hector_quadrotor_urdf/urdf/quadrotor_base.urdf.xacro (robot description, xacro)
@@ -5,5 +5,5 @@
 xmlns:xacro="http://ros.org/wiki/xacro"
 >
-  <include filename="$(find hector_quadrotor_urdf)/urdf/sonar_sensor.urdf.xacro" />
+  <include filename="$(find hector_sensors_description)/urdf/sonar_sensor.urdf.xacro" />
   <property name="pi" value="3.1415926535897931" />
   <xacro:macro name="quadrotor_base_macro">
@@ -134,5 +134,5 @@
     <!-- Sonar height sensor -->
     <sonar_sensor name="sonar" parent="base_link" ros_topic="sonar_height" update_rate="10" min_range="0.03" max_range="3.0" field_of_view="40" ray_count="3">
-      <origin xyz="0.12 0.0 -0.02" rpy="0 ${90*pi/180} 0"/>
+      <origin xyz="0.12 0.0 -0.012" rpy="0 ${90*pi/180} 0"/>
     </sonar_sensor>
   </xacro:macro>

Commit message: [hector_quadrotor_urdf] -use stl mesh for collision checking, as this does not partition into different collision objects like with COLLADA when using different materials

File: hector_quadrotor/hector_quadrotor_urdf/urdf/quadrotor_base.urdf.xacro (robot description, xacro)
@@ -17,5 +17,5 @@
         <origin xyz="0 0 0" rpy="0 0 0" />
         <geometry>
-                <mesh filename="package://hector_quadrotor_urdf/meshes/quadrotor/quadrotor_base.dae"/>
+          <mesh filename="package://hector_quadrotor_urdf/meshes/quadrotor/quadrotor_base.dae"/>
         </geometry>
       </visual>
@@ -23,5 +23,5 @@
         <origin xyz="0 0 0" rpy="0 0 0" />
         <geometry>
-          <mesh filename="package://hector_quadrotor_urdf/meshes/quadrotor/quadrotor_base.dae"/>
+          <mesh filename="package://hector_quadrotor_urdf/meshes/quadrotor/quadrotor_base.stl"/>
         </geometry>
       </collision>

Commit message: [hector_quadrotor] -minor updates to xacro files

File: hector_quadrotor/hector_quadrotor_urdf/urdf/quadrotor_base.urdf.xacro (robot description, xacro)
@@ -7,4 +7,5 @@
   <include filename="$(find hector_sensors_description)/urdf/sonar_sensor.urdf.xacro" />
   <property name="pi" value="3.1415926535897931" />
+  <!-- Main quadrotor link -->
   <xacro:macro name="quadrotor_base_macro">
     <link name="base_link">
@@ -27,7 +28,12 @@
       </collision>
     </link>
+    <!-- Sonar height sensor -->
+    <sonar_sensor name="sonar" parent="base_link" ros_topic="sonar_height" update_rate="10" min_range="0.03" max_range="3.0" field_of_view="40" ray_count="3">
+      <origin xyz="0.12 0.0 -0.012" rpy="0 ${90*pi/180} 0"/>
+    </sonar_sensor>
     <gazebo reference="base_link">
       <turnGravityOff>false</turnGravityOff>
     </gazebo>
+    <!-- Gazebo Plugins -->
     <gazebo>
       <canonicalBody>base_link</canonicalBody>
@@ -135,8 +141,4 @@
       </controller:gazebo_ros_p3d>
     </gazebo>
-    <!-- Sonar height sensor -->
-    <sonar_sensor name="sonar" parent="base_link" ros_topic="sonar_height" update_rate="10" min_range="0.03" max_range="3.0" field_of_view="40" ray_count="3">
-      <origin xyz="0.12 0.0 -0.012" rpy="0 ${90*pi/180} 0"/>
-    </sonar_sensor>
   </xacro:macro>
 </robot>

File: hector_quadrotor/hector_quadrotor_urdf/urdf/quadrotor_hokuyo_utm30lx.urdf.xacro (robot description, xacro)
@@ -10,8 +10,10 @@
     <!-- Instantiate quadrotor_base_macro once (has no parameters atm) -->
     <quadrotor_base_macro />
+    <!-- Hokuyo UTM-30LX mounted upside down below the quadrotor body -->
     <include filename="$(find hector_sensors_description)/urdf/hokuyo_utm30lx.urdf.xacro" />
     <xacro:hokuyo_utm30lx name="laser0" parent="base_link" ros_topic="scan" update_rate="40" ray_count="1081" min_angle="135" max_angle="-135">
       <origin xyz="0.0 0.0 -0.097" rpy="${M_PI} 0 0"/>
     </xacro:hokuyo_utm30lx>
+    <!-- Forward facing camera -->
     <include filename="$(find hector_sensors_description)/urdf/generic_camera.urdf.xacro" />
     <xacro:generic_camera name="front_cam" parent="base_link" ros_topic="camera/image" cam_info_topic="camera/camera_info" update_rate="10">

Commit message: hector_uav_msgs: added new package hector_quadrotor_gazebo_plugins: now uses hector_uav_msgs/Altimeter to output altimeter data (pressure, altitude and QNH) hector_quadrotor_urdf: updated sensor noise parameters and added quadrotor aerodynamics plugin

File: hector_quadrotor/hector_quadrotor_urdf/urdf/quadrotor_base.urdf.xacro (robot description, xacro)
@@ -11,7 +11,7 @@
     <link name="base_link">
       <inertial>
-        <mass value="1.316" />
+        <mass value="1.477" />
         <origin xyz="0 0 0" />
-        <inertia ixx="0.0128" ixy="0.0" ixz="0.0" iyy="0.0128" iyz="0.0" izz="0.0218" />
+        <inertia ixx="0.01152" ixy="0.0" ixz="0.0" iyy="0.01152" iyz="0.0" izz="0.0218" />
       </inertial>
       <visual>
@@ -38,18 +38,62 @@
     <gazebo>
       <canonicalBody>base_link</canonicalBody>
-      <controller:gazebo_ros_force name="gazebo_ros_force" plugin="libgazebo_ros_force.so">
+      <controller:hector_gazebo_ros_imu name="quadrotor_imu_sim" plugin="libhector_gazebo_ros_imu.so">
         <alwaysOn>true</alwaysOn>
-        <updateRate>0.0</updateRate>
+        <updateRate>100.0</updateRate>
         <bodyName>base_link</bodyName>
-        <topicName>force</topicName>
-      </controller:gazebo_ros_force>
+        <topicName>raw_imu</topicName>
+        <rpyOffsets>0 0 0</rpyOffsets> <!-- deprecated -->
+        <gaussianNoise>0</gaussianNoise>  <!-- deprecated -->
+        <accelDrift>0.5 0.5 0.5</accelDrift>
+        <accelGaussianNoise>0.35 0.35 0.3</accelGaussianNoise>
+        <rateDrift>0.1 0.1 0.1</rateDrift>
+        <rateGaussianNoise>0.05 0.05 0.015</rateGaussianNoise>
+        <headingDrift>0.1</headingDrift>
+        <headingGaussianNoise>0.05</headingGaussianNoise>
+      </controller:hector_gazebo_ros_imu>
+      <controller:hector_gazebo_ros_baro name="quadrotor_baro_sim" plugin="libhector_gazebo_ros_baro.so">
+        <alwaysOn>true</alwaysOn>
+        <updateRate>10.0</updateRate>
+        <bodyName>base_link</bodyName>
+        <topicName>pressure_height</topicName>
+        <altimeterTopicName>altimeter</altimeterTopicName>
+        <offset>0</offset>
+        <drift>0.1</drift>
+        <gaussianNoise>0.5</gaussianNoise>
+      </controller:hector_gazebo_ros_baro>
+      <controller:hector_gazebo_ros_magnetic name="quadrotor_magnetic_sim" plugin="libhector_gazebo_ros_magnetic.so">
+        <alwaysOn>true</alwaysOn>
+        <updateRate>10.0</updateRate>
+        <bodyName>base_link</bodyName>
+        <topicName>magnetic</topicName>
+        <offset>0 0 0</offset>
+        <drift>0.0 0.0 0.0</drift>
+        <gaussianNoise>1.3e-2 1.3e-2 1.3e-2</gaussianNoise>
+      </controller:hector_gazebo_ros_magnetic>
+      <controller:hector_gazebo_ros_gps name="quadrotor_gps_sim" plugin="libhector_gazebo_ros_gps.so">
+        <alwaysOn>true</alwaysOn>
+        <updateRate>4.0</updateRate>
+        <bodyName>base_link</bodyName>
+        <topicName>fix</topicName>
+        <velocityTopicName>fix_velocity</velocityTopicName>
+        <drift>5.0 5.0 5.0</drift>
+        <gaussianNoise>0.1 0.1 0.1</gaussianNoise>
+        <velocityDrift>0 0 0</velocityDrift>
+        <velocityGaussianNoise>0.1 0.1 0.1</velocityGaussianNoise>
+      </controller:hector_gazebo_ros_gps>
+      <controller:gazebo_ros_p3d name="quadrotor_groundtruth_sim" plugin="libgazebo_ros_p3d.so">
+        <alwaysOn>true</alwaysOn>
+        <updateRate>100.0</updateRate>
+        <bodyName>base_link</bodyName>
+        <topicName>ground_truth/state</topicName>
+        <gaussianNoise>0.0</gaussianNoise>
+        <frameName>map</frameName>
+      </controller:gazebo_ros_p3d>
       <controller:hector_gazebo_quadrotor_simple_controller name="quadrotor_simple_controller" plugin="libhector_gazebo_quadrotor_simple_controller.so">
         <alwaysOn>true</alwaysOn>
         <updateRate>0.0</updateRate>
         <bodyName>base_link</bodyName>
-        <!--
-          <stateTopic>ground_truth/state</stateTopic>
-          <imuTopic>raw_imu</imuTopic>
-        -->
+        <stateTopic>ground_truth/state</stateTopic>
+        <imuTopic>raw_imu</imuTopic>
         <topicName>cmd_vel</topicName>
         <rollpitch>
@@ -75,55 +119,14 @@
         <maxForce>30</maxForce>
       </controller:hector_gazebo_quadrotor_simple_controller>
-      <controller:hector_gazebo_ros_imu name="quadrotor_imu_sim" plugin="libhector_gazebo_ros_imu.so">
+      <controller:hector_gazebo_quadrotor_aerodynamics name="quadrotor_aerodynamics" plugin="libhector_gazebo_quadrotor_aerodynamics.so">
         <alwaysOn>true</alwaysOn>
-        <updateRate>100.0</updateRate>
+        <updateRate>0.0</updateRate>
         <bodyName>base_link</bodyName>
-        <topicName>raw_imu</topicName>
-        <rpyOffsets>0 0 0</rpyOffsets> <!-- deprecated -->
-        <gaussianNoise>0</gaussianNoise>  <!-- deprecated -->
-        <accelDrift>0.5 0.5 0.5</accelDrift>
-        <accelGaussianNoise>0.1 0.1 0.1</accelGaussianNoise>
-        <rateDrift>0.1 0.1 0.1</rateDrift>
-        <rateGaussianNoise>0.05 0.05 0.05</rateGaussianNoise>
-        <headingDrift>0.1</headingDrift>
-        <headingGaussianNoise>0.05</headingGaussianNoise>
-      </controller:hector_gazebo_ros_imu>
-      <controller:hector_gazebo_ros_baro name="quadrotor_baro_sim" plugin="libhector_gazebo_ros_baro.so">
-        <alwaysOn>true</alwaysOn>
-        <updateRate>10.0</updateRate>
-        <bodyName>base_link</bodyName>
-        <topicName>pressure_height</topicName>
-        <offset>0</offset>
-        <drift>0.1</drift>
-        <gaussianNoise>0.1</gaussianNoise>
-      </controller:hector_gazebo_ros_baro>
-      <controller:hector_gazebo_ros_magnetic name="quadrotor_magnetic_sim" plugin="libhector_gazebo_ros_magnetic.so">
-        <alwaysOn>true</alwaysOn>
-        <updateRate>10.0</updateRate>
-        <bodyName>base_link</bodyName>
-        <topicName>magnetic</topicName>
-        <offset>0 0 0</offset>
-        <drift>0.1 0.1 0.1</drift>
-        <gaussianNoise>0.1 0.1 0.1</gaussianNoise>
-      </controller:hector_gazebo_ros_magnetic>
-      <controller:hector_gazebo_ros_gps name="quadrotor_gps_sim" plugin="libhector_gazebo_ros_gps.so">
-        <alwaysOn>true</alwaysOn>
-        <updateRate>4.0</updateRate>
-        <bodyName>base_link</bodyName>
-        <topicName>fix</topicName>
-        <velocityTopicName>gps_velocity</velocityTopicName>
-        <drift>5.0 5.0 5.0</drift>
-        <gaussianNoise>0.1 0.1 0.1</gaussianNoise>
-        <velocityDrift>0 0 0</velocityDrift>
-        <velocityGaussianNoise>0.1 0.1 0.1</velocityGaussianNoise>
-      </controller:hector_gazebo_ros_gps>
-      <controller:gazebo_ros_p3d name="quadrotor_groundtruth_sim" plugin="libgazebo_ros_p3d.so">
-        <alwaysOn>true</alwaysOn>
-        <updateRate>100.0</updateRate>
-        <bodyName>base_link</bodyName>
-        <topicName>ground_truth/state</topicName>
-        <gaussianNoise>0.0</gaussianNoise>
-        <frameName>map</frameName>
-      </controller:gazebo_ros_p3d>
+        <topicName>motor_pwm</topicName>
+        <!--
+          <controlRate>100</controlRate>
+          <controlDelay>0.015</controlDelay>
+        -->
+      </controller:hector_gazebo_quadrotor_aerodynamics>
     </gazebo>
   </xacro:macro>

Commit message: hector_quadrotor: moved package hector_quadrotor_controller back to hector_quadrotor stack hector_quadrotor_controller: only build the aerodynamics model if Matlab is available and the model can be built hector_quadrotor_urdf: moved gazebo plugin description to hector_quadrotor_controller/urdf

File: hector_quadrotor/hector_quadrotor_urdf/urdf/quadrotor_base.urdf.xacro (robot description, xacro)
@@ -6,4 +6,5 @@
 >
   <include filename="$(find hector_sensors_description)/urdf/sonar_sensor.urdf.xacro" />
+  <include filename="$(find hector_quadrotor_controller)/urdf/quadrotor_plugins.urdf.xacro" />
   <property name="pi" value="3.1415926535897931" />
   <!-- Main quadrotor link -->
@@ -36,95 +37,5 @@
     </gazebo>
     <!-- Gazebo Plugins -->
-    <gazebo>
-      <canonicalBody>base_link</canonicalBody>
-      <controller:hector_gazebo_ros_imu name="quadrotor_imu_sim" plugin="libhector_gazebo_ros_imu.so">
-        <alwaysOn>true</alwaysOn>
-        <updateRate>100.0</updateRate>
-        <bodyName>base_link</bodyName>
-        <topicName>raw_imu</topicName>
-        <rpyOffsets>0 0 0</rpyOffsets> <!-- deprecated -->
-        <gaussianNoise>0</gaussianNoise>  <!-- deprecated -->
-        <accelDrift>0.5 0.5 0.5</accelDrift>
-        <accelGaussianNoise>0.35 0.35 0.3</accelGaussianNoise>
-        <rateDrift>0.1 0.1 0.1</rateDrift>
-        <rateGaussianNoise>0.05 0.05 0.015</rateGaussianNoise>
-        <headingDrift>0.1</headingDrift>
-        <headingGaussianNoise>0.05</headingGaussianNoise>
-      </controller:hector_gazebo_ros_imu>
-      <controller:hector_gazebo_ros_baro name="quadrotor_baro_sim" plugin="libhector_gazebo_ros_baro.so">
-        <alwaysOn>true</alwaysOn>
-        <updateRate>10.0</updateRate>
-        <bodyName>base_link</bodyName>
-        <topicName>pressure_height</topicName>
-        <altimeterTopicName>altimeter</altimeterTopicName>
-        <offset>0</offset>
-        <drift>0.1</drift>
-        <gaussianNoise>0.5</gaussianNoise>
-      </controller:hector_gazebo_ros_baro>
-      <controller:hector_gazebo_ros_magnetic name="quadrotor_magnetic_sim" plugin="libhector_gazebo_ros_magnetic.so">
-        <alwaysOn>true</alwaysOn>
-        <updateRate>10.0</updateRate>
-        <bodyName>base_link</bodyName>
-        <topicName>magnetic</topicName>
-        <offset>0 0 0</offset>
-        <drift>0.0 0.0 0.0</drift>
-        <gaussianNoise>1.3e-2 1.3e-2 1.3e-2</gaussianNoise>
-      </controller:hector_gazebo_ros_magnetic>
-      <controller:hector_gazebo_ros_gps name="quadrotor_gps_sim" plugin="libhector_gazebo_ros_gps.so">
-        <alwaysOn>true</alwaysOn>
-        <updateRate>4.0</updateRate>
-        <bodyName>base_link</bodyName>
-        <topicName>fix</topicName>
-        <velocityTopicName>fix_velocity</velocityTopicName>
-        <drift>5.0 5.0 5.0</drift>
-        <gaussianNoise>0.1 0.1 0.1</gaussianNoise>
-        <velocityDrift>0 0 0</velocityDrift>
-        <velocityGaussianNoise>0.1 0.1 0.1</velocityGaussianNoise>
-      </controller:hector_gazebo_ros_gps>
-      <controller:gazebo_ros_p3d name="quadrotor_groundtruth_sim" plugin="libgazebo_ros_p3d.so">
-        <alwaysOn>true</alwaysOn>
-        <updateRate>100.0</updateRate>
-        <bodyName>base_link</bodyName>
-        <topicName>ground_truth/state</topicName>
-        <gaussianNoise>0.0</gaussianNoise>
-        <frameName>map</frameName>
-      </controller:gazebo_ros_p3d>
-      <controller:hector_gazebo_quadrotor_simple_controller name="quadrotor_simple_controller" plugin="libhector_gazebo_quadrotor_simple_controller.so">
-        <alwaysOn>true</alwaysOn>
-        <updateRate>0.0</updateRate>
-        <bodyName>base_link</bodyName>
-        <stateTopic>ground_truth/state</stateTopic>
-        <imuTopic>raw_imu</imuTopic>
-        <topicName>cmd_vel</topicName>
-        <rollpitch>
-          <proportionalGain>10.0</proportionalGain>
-          <differentialGain>5.0</differentialGain>
-          <limit>0.5</limit>
-        </rollpitch>
-        <yaw>
-          <proportionalGain>2.0</proportionalGain>
-          <differentialGain>1.0</differentialGain>
-          <limit>1.5</limit>
-        </yaw>
-        <velocity_xy>
-          <proportionalGain>5.0</proportionalGain>
-          <differentialGain>1.0</differentialGain>
-          <limit>2</limit>
-        </velocity_xy>
-        <velocity_z>
-          <proportionalGain>5.0</proportionalGain>
-          <differentialGain>1.0</differentialGain>
-          <limit>2</limit>
-        </velocity_z>
-        <maxForce>30</maxForce>
-      </controller:hector_gazebo_quadrotor_simple_controller>
-      <!--
-      <controller:hector_gazebo_quadrotor_aerodynamics name="quadrotor_aerodynamics" plugin="libhector_gazebo_quadrotor_aerodynamics.so">
-        <alwaysOn>true</alwaysOn>
-        <updateRate>0.0</updateRate>
-        <bodyName>base_link</bodyName>
-      </controller:hector_gazebo_quadrotor_aerodynamics>
-      -->
-    </gazebo>
+    <quadrotor_plugins/>
   </xacro:macro>
 </robot>
