Commit message: [hector_xacro_tools] -remove link properties for optical frame as they don't make sense to use

File: hector_models/hector_xacro_tools/urdf/sensor_macros.urdf.xacro (robot description, xacro)
@@ -11,5 +11,5 @@
     </joint>
     <link name="${name}_optical_frame">
-      <inertial>
+<!--      <inertial>
         <mass value="0.01" />
         <origin xyz="0 0 0" />
@@ -29,5 +29,5 @@
           <box size="0.001 0.001 0.001" />
         </geometry>
-      </collision>
+      </collision>-->
     </link>
 </macro>
