Commit message: [hector_sensors_description] -thermal cam uses new mesh as used on current Hector UGV

File: hector_models/hector_sensors_description/urdf/thermaleye_camera.urdf.xacro (robot description, xacro)
@@ -18,5 +18,5 @@
           <origin xyz="0 0 0" rpy="0 0 0" />
           <geometry>
-            <mesh filename="package://hector_sensors_description/meshes/thermaleye_camera/thermaleye_camera_hector_v1.dae"/>
+            <mesh filename="package://hector_sensors_description/meshes/thermaleye_camera/thermaleye_camera_hector_v2.dae"/>
           </geometry>
         </visual>
@@ -24,5 +24,5 @@
           <origin xyz="0 0 0" rpy="0 0 0" />
           <geometry>
-            <mesh filename="package://hector_sensors_description/meshes/thermaleye_camera/thermaleye_camera_hector_v1.stl"/>
+            <mesh filename="package://hector_sensors_description/meshes/thermaleye_camera/thermaleye_camera_hector_v2.stl"/>
           </geometry>
         </collision>
