Commit message: [hector_sensors_description/hokuyo_utm30lx] -use _frame suffix for coordinate system used by sensor data. -use .stl as collision model

File: hector_models/hector_sensors_description/urdf/hokuyo_utm30lx.urdf.xacro (robot description, xacro)
@@ -9,7 +9,7 @@
 	<insert_block name="origin" />
 	<parent link="${parent}"/>
-	<child link="${name}_link"/>
+	<child link="${name}_frame"/>
       </joint>
-      <link name="${name}_link">
+      <link name="${name}_frame">
 	<inertial>
 	  <mass value="0.001" />
@@ -26,9 +26,9 @@
 	  <origin xyz="0 0 0" rpy="0 0 0" />
           <geometry>
-          <mesh filename="package://hector_sensors_description/meshes/hokuyo_utm30lx/hokuyo_utm_30lx.dae"/>
+          <mesh filename="package://hector_sensors_description/meshes/hokuyo_utm30lx/hokuyo_utm_30lx.stl"/>
         </geometry>
 	</collision>
       </link>
-      <gazebo reference="${name}_link">
+      <gazebo reference="${name}_frame">
 	<sensor:ray name="${name}">
 		<rayCount>${ray_count}</rayCount>
@@ -46,5 +46,5 @@
 	    <updateRate>${update_rate}</updateRate>
 	    <topicName>${ros_topic}</topicName>
-	    <frameName>/${name}_link</frameName>
+	    <frameName>/${name}_frame</frameName>
 	    <interface:laser name="gazebo_ros_${name}_iface" />
 	  </controller:gazebo_ros_laser>

Commit message: [hector_sensors_description] -use box model for utm30lx collision model

File: hector_models/hector_sensors_description/urdf/hokuyo_utm30lx.urdf.xacro (robot description, xacro)
@@ -24,7 +24,8 @@
 	</visual>
 	<collision>
-	  <origin xyz="0 0 0" rpy="0 0 0" />
+	  <origin xyz="0 0 -0.0115" rpy="0 0 0" />
           <geometry>
-          <mesh filename="package://hector_sensors_description/meshes/hokuyo_utm30lx/hokuyo_utm_30lx.stl"/>
+          <box size="0.058 0.058 0.087" />
+          <!--<mesh filename="package://hector_sensors_description/meshes/hokuyo_utm30lx/hokuyo_utm_30lx.stl"/>-->
         </geometry>
 	</collision>

Commit message: [hector_sensors_description] -add hokuyo utm-30lx mesh and xacro edit for TEST_SELF_FILTER in gazebo

File: hector_models/hector_sensors_description/urdf/hokuyo_utm30lx.urdf.xacro (robot description, xacro)
@@ -20,5 +20,5 @@
 	  <origin xyz="0 0 0" rpy="0 0 0" />
           <geometry>
-          <mesh filename="package://hector_sensors_description/meshes/hokuyo_utm30lx/hokuyo_utm_30lx.dae"/>
+          <mesh filename="package://hector_sensors_description/meshes/hokuyo_utm30lx/hokuyo_utm_30lx$(optenv TEST_SELF_FILTER).dae"/>
         </geometry>
 	</visual>
