Commit message: [hector_sensors_description] -change generic_camera macro to include resolution, hfov and image format as parameters

File: hector_models/hector_sensors_description/urdf/generic_camera.urdf.xacro (robot description, xacro)
@@ -6,5 +6,5 @@
   >
     <property name="M_PI" value="3.1415926535897931" />
-    <xacro:macro name="generic_camera" params="name parent *origin ros_topic cam_info_topic update_rate">
+    <xacro:macro name="generic_camera" params="name parent *origin ros_topic cam_info_topic update_rate res_x res_y image_format hfov">
       <joint name="${name}_joint" type="fixed">
         <insert_block name="origin" />
@@ -62,7 +62,7 @@
     <gazebo reference="${name}_link">
       <sensor:camera name="${name}_camera_sensor">
-        <imageSize>320 240</imageSize>
-        <imageFormat>R8G8B8</imageFormat>
-        <hfov>90</hfov>
+        <imageSize>${res_x} ${res_y}</imageSize>
+        <imageFormat>${image_format}</imageFormat>
+        <hfov>${hfov}</hfov>
         <nearClip>0.01</nearClip>
         <farClip>100</farClip>

File: hector_quadrotor/hector_quadrotor_urdf/urdf/quadrotor_downward_cam.xacro (robot description, xacro)
@@ -11,12 +11,12 @@
     <quadrotor_base_macro />
     <!-- Hokuyo UTM-30LX mounted upside down below the quadrotor body -->
-    <include filename="$(find hector_sensors_description)/urdf/hokuyo_utm30lx.urdf.xacro" />
+<!--    <include filename="$(find hector_sensors_description)/urdf/hokuyo_utm30lx.urdf.xacro" />
     <xacro:hokuyo_utm30lx name="laser0" parent="base_link" ros_topic="scan" update_rate="40" ray_count="1081" min_angle="135" max_angle="-135">
       <origin xyz="0.0 0.0 -0.097" rpy="${M_PI} 0 0"/>
-    </xacro:hokuyo_utm30lx>
+    </xacro:hokuyo_utm30lx>-->
     <!-- Forward facing camera -->
     <include filename="$(find hector_sensors_description)/urdf/generic_camera.urdf.xacro" />
-    <xacro:generic_camera name="front_cam" parent="base_link" ros_topic="camera/image" cam_info_topic="camera/camera_info" update_rate="10" res_x="320" res_y="240" image_format="R8G8B8" hfov="90">
-      <origin xyz="0.05 0.0 -0.06" rpy="0 0 0"/>
+    <xacro:generic_camera name="downward_cam" parent="base_link" ros_topic="camera/image" cam_info_topic="camera/camera_info" update_rate="20" res_x="640" res_y="480" image_format="L8" hfov="100">
+      <origin xyz="0.4 0.0 -0.0" rpy="0 ${M_PI/2} 0"/>
     </xacro:generic_camera>
 </robot>
