Commit message: merged updates from /branches/fuerte

File: hector_models/hector_sensors_description/urdf/asus_camera.urdf.xacro (robot description, xacro)
@@ -7,5 +7,5 @@
     <include filename="$(find hector_xacro_tools)/urdf/sensor_macros.urdf.xacro" />
     <property name="M_PI" value="3.1415926535897931" />
-    <xacro:macro name="kinect_camera_model" params="name parent *origin">
+    <xacro:macro name="asus_camera_model" params="name parent *origin">
       <joint name="${name}_joint" type="fixed">
         <insert_block name="origin" />
@@ -14,9 +14,13 @@
       </joint>
       <link name="${name}_link">
-        <inertial_sphere mass="0.01" diameter="0.07" />
+        <inertial>
+	  <mass value="0.200" />
+	  <origin xyz="0 0 0" rpy="0 0 0" />
+		<inertia ixx="5.8083e-4" ixy="0" ixz="0" iyy="3.0833e-5" iyz="0" izz="5.9083e-4" />
+	</inertial>
         <visual>
           <origin xyz="0 0 0" rpy="0 0 0" />
           <geometry>
-            <mesh filename="package://hector_sensors_description/meshes/kinect_camera/kinect_camera_simple.dae"/>
+            <mesh filename="package://hector_sensors_description/meshes/asus_camera/asus_camera_simple.dae"/>
           </geometry>
         </visual>
@@ -24,10 +28,10 @@
           <origin xyz="0 0 0" rpy="0 0 0" />
           <geometry>
-            <mesh filename="package://hector_sensors_description/meshes/kinect_camera/kinect_camera_simple.stl"/>
+            <box size="0.035 0.185 0.025"/>
           </geometry>
         </collision>
       </link>
       <joint name="${name}_depth_joint" type="fixed">
-        <origin xyz="0.0 -0.02 0.0" rpy="0 0 0" />
+        <origin xyz="0.0 0.049 0.0" rpy="0 0 0" />
         <parent link="${name}_link" />
         <child link="${name}_depth_frame"/>
@@ -41,5 +45,5 @@
       <link name="${name}_depth_optical_frame"/>
       <joint name="${name}_rgb_joint" type="fixed">
-        <origin xyz="0.0 -0.045 0.0" rpy="0 0 0" />
+        <origin xyz="0.0 0.022 0.0" rpy="0 0 0" />
         <parent link="${name}_link" />
         <child link="${name}_rgb_frame"/>
@@ -53,42 +57,16 @@
       <link name="${name}_rgb_optical_frame"/>
     </xacro:macro>
-    <xacro:macro name="kinect_camera" params="name parent *origin">
-      <kinect_camera_model name="${name}" parent="${parent}">
+    <xacro:macro name="asus_camera" params="name parent *origin">
+      <asus_camera_model name="${name}" parent="${parent}">
         <insert_block name="origin" />
-      </kinect_camera_model>
+      </asus_camera_model>
       <!-- ASUS Xtion PRO camera for simulation -->
-      <!-- gazebo_ros_wge100 plugin is in kt2_gazebo_plugins package -->
-      <!-- <gazebo reference="${name}_link" >
-        <sensor:camera name="${name}" >
-          <imageSize>640 480</imageSize>
-          <imageFormat>R8G8B8</imageFormat>
-          <hfov>62.8</hfov>
-          <nearClip>0.1</nearClip>
-          <farClip>10</farClip>
-          <updateRate>2.0</updateRate>
-          <controller:gazebo_ros_wge100 name="${name}_camera_controller" plugin="libgazebo_ros_wge100.so">
-	    <alwaysOn>true</alwaysOn>
-	    <updateRate>5000.0</updateRate>
-	    <cameraName>${name}/rgb</cameraName>
-	    <frameName>${name}_rgb_optical_frame</frameName>
-	    <hackBaseline>0.0</hackBaseline>
-	    <CxPrime>320.5</CxPrime>
-	    <Cx>320.5</Cx>
-	    <Cy>240.5</Cy>
-	    <baseline>0.09</baseline>
-	    <focal_length>525</focal_length>
-	    <cameraNamespace>camera/rgb</cameraNamespace>
-	    <depthData>true</depthData>
-	    <interface:camera name="camera_iface" />
-          </controller:gazebo_ros_wge100>
-        </sensor:camera>
-      </gazebo> -->
       <gazebo reference="${name}_depth_frame">
         <sensor:camera name="${name}">
           <imageFormat>R8G8B8</imageFormat>
           <imageSize>640 480</imageSize>
-          <hfov>60</hfov>
-          <nearClip>0.05</nearClip>
-          <farClip>3</farClip>
+          <hfov>62.8</hfov>
+          <nearClip>0.5</nearClip>
+          <farClip>9</farClip>
           <updateRate>20</updateRate>
           <baseline>0.1</baseline>

File: hector_models/hector_sensors_description/urdf/generic_camera.urdf.xacro (robot description, xacro)
@@ -39,25 +39,5 @@
       <child link="${name}_optical_frame"/>
     </joint>
-    <link name="${name}_optical_frame">
-      <inertial>
-        <mass value="0.01" />
-        <origin xyz="0 0 0" />
-        <inertia ixx="0.001"  ixy="0.0"  ixz="0.0"
-                 iyy="0.001"  iyz="0.0"
-                 izz="0.001" />
-      </inertial>
-      <visual>
-        <origin xyz="0 0 0" rpy="0 0 0"/>
-        <geometry>
-          <box size="0.001 0.001 0.001" />
-        </geometry>
-      </visual>
-      <collision>
-        <origin xyz="0 0 0" rpy="0 0 0"/>
-        <geometry>
-          <box size="0.001 0.001 0.001" />
-        </geometry>
-      </collision>
-    </link>
+    <link name="${name}_optical_frame"/>
     <gazebo reference="${name}_link">
       <sensor:camera name="${name}_camera_sensor">

File: hector_models/hector_sensors_description/urdf/hokuyo_utm30lx.urdf.xacro (robot description, xacro)
@@ -13,7 +13,7 @@
       <link name="${name}_frame">
 	<inertial>
-	  <mass value="0.001" />
+	  <mass value="0.270" />
 	  <origin xyz="0 0 0" rpy="0 0 0" />
-		<inertia ixx="0.0001" ixy="0" ixz="0" iyy="0.0001" iyz="0" izz="0.0001" />
+		<inertia ixx="2.632e-4" ixy="0" ixz="0" iyy="2.632e-4" iyz="0" izz="1.62e-4" />
 	</inertial>
 	<visual>

File: hector_quadrotor/hector_quadrotor_urdf/urdf/quadrotor_base.urdf.xacro (robot description, xacro)
@@ -31,5 +31,5 @@
     <!-- Sonar height sensor -->
     <sonar_sensor name="sonar" parent="base_link" ros_topic="sonar_height" update_rate="10" min_range="0.03" max_range="3.0" field_of_view="40" ray_count="3">
-      <origin xyz="0.12 0.0 -0.012" rpy="0 ${90*pi/180} 0"/>
+      <origin xyz="-0.16 0.0 -0.012" rpy="0 ${90*pi/180} 0"/>
     </sonar_sensor>
     <gazebo reference="base_link">

Commit message: hector_models: cleaned up urdf and bumped version to 0.1.1

File: hector_models/hector_sensors_description/urdf/asus_camera.urdf.xacro (robot description, xacro)
@@ -15,8 +15,8 @@
       <link name="${name}_link">
         <inertial>
-	  <mass value="0.200" />
-	  <origin xyz="0 0 0" rpy="0 0 0" />
-		<inertia ixx="5.8083e-4" ixy="0" ixz="0" iyy="3.0833e-5" iyz="0" izz="5.9083e-4" />
-	</inertial>
+          <mass value="0.200" />
+          <origin xyz="0 0 0" rpy="0 0 0" />
+          <inertia ixx="5.8083e-4" ixy="0" ixz="0" iyy="3.0833e-5" iyz="0" izz="5.9083e-4" />
+        </inertial>
         <visual>
           <origin xyz="0 0 0" rpy="0 0 0" />

File: hector_models/hector_sensors_description/urdf/hokuyo_utm30lx.urdf.xacro (robot description, xacro)
@@ -7,51 +7,51 @@
     <xacro:macro name="hokuyo_utm30lx" params="name parent *origin ros_topic update_rate ray_count min_angle max_angle">
       <joint name="${name}_joint" type="fixed">
-	<insert_block name="origin" />
-	<parent link="${parent}"/>
-	<child link="${name}_frame"/>
+        <insert_block name="origin" />
+        <parent link="${parent}"/>
+        <child link="${name}_frame"/>
       </joint>
-<link name="${name}_frame">
-	<inertial>
-	  <mass value="0.270" />
-	  <origin xyz="0 0 0" rpy="0 0 0" />
-		<inertia ixx="2.632e-4" ixy="0" ixz="0" iyy="2.632e-4" iyz="0" izz="1.62e-4" />
-	</inertial>
-	<visual>
-	  <origin xyz="0 0 0" rpy="0 0 0" />
+      <link name="${name}_frame">
+        <inertial>
+          <mass value="0.270" />
+          <origin xyz="0 0 0" rpy="0 0 0" />
+          <inertia ixx="2.632e-4" ixy="0" ixz="0" iyy="2.632e-4" iyz="0" izz="1.62e-4" />
+        </inertial>
+        <visual>
+          <origin xyz="0 0 0" rpy="0 0 0" />
           <geometry>
           <mesh filename="package://hector_sensors_description/meshes/hokuyo_utm30lx/hokuyo_utm_30lx$(optenv TEST_SELF_FILTER).dae"/>
         </geometry>
-	</visual>
-	<collision>
-	  <origin xyz="0 0 -0.0115" rpy="0 0 0" />
+        </visual>
+        <collision>
+          <origin xyz="0 0 -0.0115" rpy="0 0 0" />
           <geometry>
           <box size="0.058 0.058 0.087" />
           <!--<mesh filename="package://hector_sensors_description/meshes/hokuyo_utm30lx/hokuyo_utm_30lx.stl"/>-->
         </geometry>
-	</collision>
-</link>
-  <gazebo reference="${name}_frame">
-    <sensor:ray name="${name}">
-    <rayCount>${ray_count}</rayCount>
-    <rangeCount>${ray_count}</rangeCount>
-        <laserCount>1</laserCount>
-        <origin>0.0 0.0 0.0</origin>
-        <displayRays>false</displayRays>
-        <minAngle>${min_angle}</minAngle>
-        <maxAngle>${max_angle}</maxAngle>
-        <minRange>0.08</minRange>
-        <maxRange>30.0</maxRange>
-        <resRange>0.01</resRange>
-        <updateRate>${update_rate}</updateRate>
-        <controller:gazebo_ros_laser name="gazebo_ros_${name}_controller" plugin="libgazebo_ros_laser.so">
-          <gaussianNoise>0.005</gaussianNoise>
-          <alwaysOn>true</alwaysOn>
+        </collision>
+      </link>
+      <gazebo reference="${name}_frame">
+        <sensor:ray name="${name}">
+          <rayCount>${ray_count}</rayCount>
+          <rangeCount>${ray_count}</rangeCount>
+          <laserCount>1</laserCount>
+          <origin>0.0 0.0 0.0</origin>
+          <displayRays>false</displayRays>
+          <minAngle>${min_angle}</minAngle>
+          <maxAngle>${max_angle}</maxAngle>
+          <minRange>0.08</minRange>
+          <maxRange>30.0</maxRange>
+          <resRange>0.01</resRange>
           <updateRate>${update_rate}</updateRate>
-          <topicName>${ros_topic}</topicName>
-          <frameName>${name}_frame</frameName>
-          <interface:laser name="gazebo_ros_${name}_iface" />
-        </controller:gazebo_ros_laser>
-      </sensor:ray>
-    </gazebo>
+          <controller:gazebo_ros_laser name="gazebo_ros_${name}_controller" plugin="libgazebo_ros_laser.so">
+            <gaussianNoise>0.005</gaussianNoise>
+            <alwaysOn>true</alwaysOn>
+            <updateRate>${update_rate}</updateRate>
+            <topicName>${ros_topic}</topicName>
+            <frameName>${name}_frame</frameName>
+            <interface:laser name="gazebo_ros_${name}_iface" />
+          </controller:gazebo_ros_laser>
+        </sensor:ray>
+      </gazebo>
     </xacro:macro>
   </robot>

File: hector_models/hector_sensors_description/urdf/kinect_camera.urdf.xacro (robot description, xacro)
@@ -57,31 +57,4 @@
         <insert_block name="origin" />
       </kinect_camera_model>
-      <!-- ASUS Xtion PRO camera for simulation -->
-      <!-- gazebo_ros_wge100 plugin is in kt2_gazebo_plugins package -->
-      <!-- <gazebo reference="${name}_link" >
-        <sensor:camera name="${name}" >
-          <imageSize>640 480</imageSize>
-          <imageFormat>R8G8B8</imageFormat>
-          <hfov>62.8</hfov>
-          <nearClip>0.1</nearClip>
-          <farClip>10</farClip>
-          <updateRate>2.0</updateRate>
-          <controller:gazebo_ros_wge100 name="${name}_camera_controller" plugin="libgazebo_ros_wge100.so">
-	    <alwaysOn>true</alwaysOn>
-	    <updateRate>5000.0</updateRate>
-	    <cameraName>${name}/rgb</cameraName>
-	    <frameName>${name}_rgb_optical_frame</frameName>
-	    <hackBaseline>0.0</hackBaseline>
-	    <CxPrime>320.5</CxPrime>
-	    <Cx>320.5</Cx>
-	    <Cy>240.5</Cy>
-	    <baseline>0.09</baseline>
-	    <focal_length>525</focal_length>
-	    <cameraNamespace>camera/rgb</cameraNamespace>
-	    <depthData>true</depthData>
-	    <interface:camera name="camera_iface" />
-          </controller:gazebo_ros_wge100>
-        </sensor:camera>
-      </gazebo> -->
       <gazebo reference="${name}_depth_frame">
         <sensor:camera name="${name}">
