Commit message: [hector_ugv_common] -temporarily comment out controllers while the model spawning crashes on fuerte

File: hector_ugv_common/hector_ugv_description/urdf/hector_ugv_base.urdf.xacro (robot description, xacro)
@@ -71,5 +71,4 @@
           <geometry>
            <mesh filename="package://hector_ugv_description/meshes/$(env ROBOT)_top_box$(optenv TEST_SELF_FILTER).dae"/>
-            <!--<box size="0.001 0.01 0.01" />-->
           </geometry>
     </visual>
@@ -77,7 +76,5 @@
       <origin xyz="${top_box_pos_x} ${top_box_pos_y} ${top_box_pos_z}" rpy="0 0 0" />
       <geometry>
-          <!--<mesh filename="package://monstertruck_urdf/meshes/$(env ROBOT)_top_box.stl"/>-->
           <box size="${top_box_size_x} ${top_box_size_y} ${top_box_size_z}" />
-          <!--<box size="0.001 0.01 0.01" />-->
       </geometry>
     </collision>
@@ -333,5 +330,5 @@
     </collision>
   </link>-->
-   <xacro:thermaleye_camera_model name="infrared" parent="mounting_link">
+<!--   <xacro:thermaleye_camera_model name="infrared" parent="mounting_link">
      <origin xyz="${infrared_x_position} ${infrared_y_position} ${infrared_z_position}" rpy="0 0 0" />
    </xacro:thermaleye_camera_model>
@@ -339,5 +336,5 @@
      <origin xyz="${kinect_x_position} 0 ${kinect_z_position}" rpy="0 0 0" />
    </xacro:kinect_camera_model>
-   <include filename="$(find monstertruck_urdf)/hector/$(env ROBOT)_addons.urdf.xacro" />
+   <include filename="$(find monstertruck_urdf)/hector/$(env ROBOT)_addons.urdf.xacro" />-->
   <hector_wheel parent="base_link" prefix="Front" suffix="left" reflect_x="1" reflect_y="1" wheel_joint_type="${wheel_joint_type}" />
   <hector_wheel parent="base_link" prefix="Front" suffix="right" reflect_x="1" reflect_y="-1" wheel_joint_type="${wheel_joint_type}" />

File: hector_ugv_common/hector_ugv_gazebo/urdf/hector_ugv.gazebo.xacro (robot description, xacro)
@@ -11,5 +11,5 @@
   <include filename="$(find hector_ugv_description)/urdf/hector_ugv_base.urdf.xacro" />
   <hector_ugv_base wheel_joint_type="continuous" />
-  <include filename="$(find hector_sensors_description)/urdf/hokuyo_utm30lx.urdf.xacro" />
+<!--  <include filename="$(find hector_sensors_description)/urdf/hokuyo_utm30lx.urdf.xacro" />
   <xacro:hokuyo_utm30lx name="laser1" parent="laser1_link" ros_topic="laser1/scan" update_rate="40" ray_count="1081" min_angle="135" max_angle="-135">
     <origin xyz="${laser1_center_x_offset} 0 ${laser1_plane_height}" rpy="0 0 0"/>
@@ -62,4 +62,4 @@
         </controller:gazebo_ros_thermal_camera>
       </sensor:camera>
-    </gazebo>
+    </gazebo>-->
 </robot>
