Commit message: [hector_ugv_common] -fixes

File: hector_ugv_common/hector_ugv_description/urdf/hector_ugv.urdf.xacro (robot description, xacro)
@@ -5,11 +5,11 @@
 	 xmlns:xacro="http://playerstage.sourceforge.net/gazebo/xmlschema/#interface"
 	 name="hector">
-  <include filename="$(find monstertruck_urdf)/hector/materials.urdf.xacro" />
-  <include filename="$(find monstertruck_urdf)/hector/hector_wheel.urdf.xacro" />
-  <include filename="$(find monstertruck_urdf)/hector/hector_ugv_common_dimensions.urdf.xacro" />
-  <include filename="$(find monstertruck_urdf)/hector/$(env ROBOT)_dimensions.urdf.xacro" />
-  <include filename="$(find monstertruck_urdf)/hector/hector_ugv_base.urdf.xacro" />
+  <include filename="$(find hector_ugv_description)/urdf/materials.urdf.xacro" />
+  <include filename="$(find hector_ugv_description)/urdf/hector_wheel.urdf.xacro" />
+  <include filename="$(find hector_ugv_description)/urdf/hector_ugv_common_dimensions.urdf.xacro" />
+  <include filename="$(find hector_ugv_description)/urdf/$(env ROBOT)_dimensions.urdf.xacro" />
+  <include filename="$(find hector_ugv_description)/urdf/hector_ugv_base.urdf.xacro" />
   <hector_ugv_base wheel_joint_type="fixed" />
-  <include filename="$(find monstertruck_urdf)/hector/hector_ugv_openni_frames.urdf.xacro" />
+  <include filename="$(find hector_ugv_description)/urdf/hector_ugv_openni_frames.urdf.xacro" />
   <include filename="$(find hector_sensors_description)/urdf/hokuyo_utm30lx.urdf.xacro" />
   <xacro:hokuyo_utm30lx name="laser1" parent="laser1_link" ros_topic="laser1/scan" update_rate="40" ray_count="1081" min_angle="135" max_angle="-135">

File: hector_ugv_common/hector_ugv_description/urdf/hector_ugv_base.urdf.xacro (robot description, xacro)
@@ -49,11 +49,11 @@
       <origin xyz="0.0 0.0 0.0" rpy="0 0 0" />
       <geometry>
-        <mesh filename="package://monstertruck_urdf/meshes/hector_common_base.dae"/>
-      </geometry>
-    </visual>
-    <collision>
-      <origin xyz="0.0 0.0 0.0" rpy="0 0 0" />
-      <geometry>
-          <mesh filename="package://monstertruck_urdf/meshes/hector_common_base.stl"/>
+        <mesh filename="package://hector_ugv_description/meshes/hector_common_base.dae"/>
+      </geometry>
+    </visual>
+    <collision>
+      <origin xyz="0.0 0.0 0.0" rpy="0 0 0" />
+      <geometry>
+          <mesh filename="package://hector_ugv_description/meshes/hector_common_base.stl"/>
       </geometry>
     </collision>
@@ -70,5 +70,5 @@
           <origin xyz="0.0 0.0 0.0" rpy="0 0 0" />
           <geometry>
-           <mesh filename="package://monstertruck_urdf/meshes/$(env ROBOT)_top_box$(optenv TEST_SELF_FILTER).dae"/>
+           <mesh filename="package://hector_ugv_description/meshes/$(env ROBOT)_top_box$(optenv TEST_SELF_FILTER).dae"/>
             <!--<box size="0.001 0.01 0.01" />-->
           </geometry>

Commit message: [hector_ugv_description] -switch off ROBOT env variable based selection of geometry for the moment.

File: hector_ugv_common/hector_ugv_description/urdf/hector_ugv.urdf.xacro (robot description, xacro)
@@ -8,5 +8,5 @@
   <include filename="$(find hector_ugv_description)/urdf/hector_wheel.urdf.xacro" />
   <include filename="$(find hector_ugv_description)/urdf/hector_ugv_common_dimensions.urdf.xacro" />
-  <include filename="$(find hector_ugv_description)/urdf/$(env ROBOT)_dimensions.urdf.xacro" />
+  <include filename="$(find hector_ugv_description)/urdf/hector1_dimensions.urdf.xacro" />
   <include filename="$(find hector_ugv_description)/urdf/hector_ugv_base.urdf.xacro" />
   <hector_ugv_base wheel_joint_type="fixed" />

File: hector_ugv_common/hector_ugv_description/urdf/hector_ugv_base.urdf.xacro (robot description, xacro)
@@ -70,5 +70,5 @@
           <origin xyz="0.0 0.0 0.0" rpy="0 0 0" />
           <geometry>
-           <mesh filename="package://hector_ugv_description/meshes/$(env ROBOT)_top_box$(optenv TEST_SELF_FILTER).dae"/>
+           <mesh filename="package://hector_ugv_description/meshes/hector1_top_box$(optenv TEST_SELF_FILTER).dae"/>
           </geometry>
     </visual>
