Commit message: [biorob_common] -renaming inside files due to name change

File: biorob_common/biorob_description/urdf/biorob_v3_x4/biorob_v3_x4.urdf.xacro (robot description, xacro)
@@ -1,9 +1,9 @@
 <?xml version="1.0"?>
-<robot name="biorob_x4"
+<robot name="biorob_v3_x4"
     xmlns:sensor="http://playerstage.sourceforge.net/gazebo/xmlschema/#sensor"
     xmlns:controller="http://playerstage.sourceforge.net/gazebo/xmlschema/#controller"
     xmlns:interface="http://playerstage.sourceforge.net/gazebo/xmlschema/#interface">
     <!-- Included URDF Files -->
-    <include filename="$(find biorob_description)/urdf/biorob_x4/biorob_x4_base.urdf.xacro" />
+    <include filename="$(find biorob_description)/urdf/biorob_x4/biorob_v3_x4_base.urdf.xacro" />
     <link name="base">
       <inertial>

File: biorob_common/biorob_description/urdf/biorob_v3_x4/biorob_v3_x4_base.urdf.xacro (robot description, xacro)
@@ -4,5 +4,5 @@
 xmlns:interface="http://playerstage.sourceforge.net/gazebo/xmlschema/#interface"
 xmlns:xacro="http://playerstage.sourceforge.net/gazebo/xmlschema/#interface"
-name="biorob_x4">
+name="biorob_v3_x4">
   <xacro:property name="base_height" value=".009"/>
   <xacro:property name="j1_length" value=".276"/>

File: biorob_common/biorob_description/urdf/biorob_v3_x4/biorob_v3_x4_base_self_filter.urdf.xacro (robot description, xacro)
@@ -4,5 +4,5 @@
 xmlns:interface="http://playerstage.sourceforge.net/gazebo/xmlschema/#interface"
 xmlns:xacro="http://playerstage.sourceforge.net/gazebo/xmlschema/#interface"
-name="biorob_x4">
+name="biorob_v3_x4">
   <xacro:property name="base_height" value=".009"/>
   <xacro:property name="j1_length" value=".276"/>

File: biorob_common/biorob_description/urdf/biorob_v3_x4/biorob_v3_x4_self_filter.urdf.xacro (robot description, xacro)
@@ -1,9 +1,9 @@
 <?xml version="1.0"?>
-<robot name="biorob_x4"
+<robot name="biorob_v3_x4"
     xmlns:sensor="http://playerstage.sourceforge.net/gazebo/xmlschema/#sensor"
     xmlns:controller="http://playerstage.sourceforge.net/gazebo/xmlschema/#controller"
     xmlns:interface="http://playerstage.sourceforge.net/gazebo/xmlschema/#interface">
     <!-- Included URDF Files -->
-    <include filename="$(find biorob_description)/urdf/biorob_x4/biorob_x4_base_self_filter.urdf.xacro" />
+    <include filename="$(find biorob_description)/urdf/biorob_x4/biorob_v3_x4_base_self_filter.urdf.xacro" />
     <link name="base">
       <inertial>

File: biorob_common/biorob_description/urdf/biorob_v3_x6/biorob_v3_x6.urdf.xacro (robot description, xacro)
@@ -1,4 +1,4 @@
 <?xml version="1.0"?>
-<robot name="biorob_x6"
+<robot name="biorob_v3_x6"
     xmlns:sensor="http://playerstage.sourceforge.net/gazebo/xmlschema/#sensor"
     xmlns:controller="http://playerstage.sourceforge.net/gazebo/xmlschema/#controller"

File: biorob_common/biorob_description/urdf/biorob_v3_x6/biorob_v3_x6_base.urdf.xacro (robot description, xacro)
@@ -1,4 +1,8 @@
 <?xml version="1.0"?>
-<robot xmlns:sensor="http://playerstage.sourceforge.net/gazebo/xmlschema/#sensor" xmlns:controller="http://playerstage.sourceforge.net/gazebo/xmlschema/#controller" xmlns:interface="http://playerstage.sourceforge.net/gazebo/xmlschema/#interface" xmlns:xacro="http://playerstage.sourceforge.net/gazebo/xmlschema/#interface" name="biorob_x4">
+<robot xmlns:sensor="http://playerstage.sourceforge.net/gazebo/xmlschema/#sensor"
+       xmlns:controller="http://playerstage.sourceforge.net/gazebo/xmlschema/#controller"
+       xmlns:interface="http://playerstage.sourceforge.net/gazebo/xmlschema/#interface"
+       xmlns:xacro="http://playerstage.sourceforge.net/gazebo/xmlschema/#interface"
+       name="biorob_v3_x6">
   <xacro:property name="base_height" value=".009"/>
   <xacro:property name="j1_length" value=".276"/>
@@ -97,5 +101,5 @@
       <visual>
         <geometry>
-          <mesh filename="package://biorob_description/meshes/biorob_x6/biorob_x6_link_3.dae"/>
+          <mesh filename="package://biorob_description/meshes/biorob_x6/biorob_v3_x6_link_3.dae"/>
           <!--<cylinder radius="0.02" length="${j3_length}" />-->
         </geometry>
@@ -106,5 +110,5 @@
       <collision>
         <geometry>
-          <mesh filename="package://biorob_description/meshes/biorob_x6/biorob_x6_link_3.dae"/>
+          <mesh filename="package://biorob_description/meshes/biorob_x6/biorob_v3_x6_link_3.dae"/>
           <!--  <cylinder radius="0.02" length="${j3_length}" />-->
         </geometry>
@@ -121,5 +125,5 @@
       <visual>
         <geometry>
-          <mesh filename="package://biorob_description/meshes/biorob_x6/biorob_x6_link_4.dae"/>
+          <mesh filename="package://biorob_description/meshes/biorob_x6/biorob_v3_x6_link_4.dae"/>
           <!--                    <cylinder radius="0.002" length="0.001" />-->
         </geometry>
@@ -130,5 +134,5 @@
       <collision>
         <geometry>
-          <mesh filename="package://biorob_description/meshes/biorob_x6/biorob_x6_link_4.dae"/>
+          <mesh filename="package://biorob_description/meshes/biorob_x6/biorob_v3_x6_link_4.dae"/>
           <!--<cylinder radius="0.02" length="${j4_length}" />-->
         </geometry>
@@ -169,5 +173,5 @@
       <visual>
         <geometry>
-          <mesh filename="package://biorob_description/meshes/biorob_x6/biorob_x6_link_6.dae"/>
+          <mesh filename="package://biorob_description/meshes/biorob_x6/biorob_v3_x6_link_6.dae"/>
           <!--<cylinder radius="0.002" length="0.001" />-->
         </geometry>
@@ -178,5 +182,5 @@
       <collision>
         <geometry>
-          <mesh filename="package://biorob_description/meshes/biorob_x6/biorob_x6_link_6.dae"/>
+          <mesh filename="package://biorob_description/meshes/biorob_x6/biorob_v3_x6_link_6.dae"/>
           <!--<cylinder radius="0.002" length="0.001" />-->
         </geometry>

File: biorob_common/biorob_gazebo/urdf/biorob_v3_x4.gazebo.xacro (robot description, xacro)
@@ -4,5 +4,5 @@
     xmlns:controller="http://playerstage.sourceforge.net/gazebo/xmlschema/#controller"
     xmlns:interface="http://playerstage.sourceforge.net/gazebo/xmlschema/#interface">
-  <include filename="$(find biorob_description)/urdf/biorob_x4/biorob_x4.urdf.xacro" />
+  <include filename="$(find biorob_description)/urdf/biorob_x4/biorob_v3_x4.urdf.xacro" />
   <gazebo>
     <controller:gazebo_ros_controller_manager name="gazebo_ros_controller_manager" plugin="libgazebo_ros_controller_manager.so">

File: biorob_common/biorob_gazebo/urdf/biorob_v3_x6.gazebo.xacro (robot description, xacro)
@@ -4,5 +4,5 @@
     xmlns:controller="http://playerstage.sourceforge.net/gazebo/xmlschema/#controller"
     xmlns:interface="http://playerstage.sourceforge.net/gazebo/xmlschema/#interface">
-  <include filename="$(find biorob_description)/urdf/biorob_x6/biorob_x6.urdf.xacro" />
+  <include filename="$(find biorob_description)/urdf/biorob_x6/biorob_v3_x6.urdf.xacro" />
   <gazebo>
     <controller:gazebo_ros_controller_manager name="gazebo_ros_controller_manager" plugin="libgazebo_ros_controller_manager.so">
