Commit message: [biorob_common] -fix toolframe translation for biorob_v3_x6

File: biorob_common/biorob_description/urdf/biorob_v3_x6/biorob_v3_x6_base.urdf.xacro (robot description, xacro)
@@ -258,5 +258,5 @@
       <child link="biorob_toolframe"/>
       <axis xyz="0 0 1"/>
-      <origin xyz="1 0.0 0.0" rpy="${-pi/2} 0 0"/>
+      <origin xyz="0.02 0.0 0.0" rpy="${-pi/2} 0 0"/>
     </joint>
     <transmission type="pr2_mechanism_model/SimpleTransmission" name="joint1_trans">
