Commit message: hector_quadrotor: - hector_quadrotor_gazebo: added cmake switch to enable/disable usage of ground truth information for the controller - hector_quadrotor_gazebo: added cmake logic to fall back to the simple controller if the required plugins for the advanced controller are not built - hector_quadrotor_controller: added urdf for the advanced quadrotor controller - hector_quadrotor_gazebo_plugins: added a workaround to circumvent a segfault in gazebo if a parameter value is empty

File: hector_quadrotor/hector_quadrotor_controller/urdf/quadrotor_propulsion.urdf.xacro (robot description, xacro)
@@ -4,5 +4,5 @@
 xmlns:xacro="http://ros.org/wiki/xacro"
 >
-  <!-- Quadrotor Aerodynamics Plugin -->
+  <!-- Quadrotor Propulsion -->
   <xacro:macro name="quadrotor_propulsion">
     <gazebo>
@@ -11,6 +11,6 @@
         <updateRate>0.0</updateRate>
         <bodyName>base_link</bodyName>
-        <controlRate>100.0</controlRate>
-        <controlDelay>0.01</controlDelay>
+        <!-- <controlRate>100.0</controlRate> -->
+        <!-- <controlDelay>0.01</controlDelay> -->
       </controller:hector_gazebo_quadrotor_propulsion>
     </gazebo>

File: hector_quadrotor/hector_quadrotor_gazebo_plugins/urdf/quadrotor_simple_controller.urdf.xacro (robot description, xacro)
@@ -5,5 +5,5 @@
 >
   <!-- Quadrotor Simple Controller Plugin -->
-  <xacro:macro name="quadrotor_simple_controller">
+  <xacro:macro name="quadrotor_simple_controller" params="state_topic imu_topic">
     <gazebo>
       <controller:hector_gazebo_quadrotor_simple_controller name="quadrotor_simple_controller" plugin="libhector_gazebo_quadrotor_simple_controller.so">
@@ -11,7 +11,7 @@
         <updateRate>0.0</updateRate>
         <bodyName>base_link</bodyName>
-        <stateTopic>ground_truth/state</stateTopic>
-        <imuTopic>raw_imu</imuTopic>
         <topicName>cmd_vel</topicName>
+        <stateTopic>${state_topic}</stateTopic>
+        <imuTopic>${imu_topic}</imuTopic>
         <rollpitchProportionalGain>10.0</rollpitchProportionalGain>
         <rollpitchDifferentialGain>5.0</rollpitchDifferentialGain>
@@ -22,5 +22,5 @@
         <velocityXYProportionalGain>5.0</velocityXYProportionalGain>
         <velocityXYDifferentialGain>1.0</velocityXYDifferentialGain>
-        <velocityXYLimit>2</velocityXYLimit>
+        <velocityXYLimit>5</velocityXYLimit>
         <velocityZProportionalGain>5.0</velocityZProportionalGain>
         <velocityZDifferentialGain>1.0</velocityZDifferentialGain>
