Commit message: hector_quadrotor_controller: - updated model parameters - added power loss in the motor controllers to the model - added trigger output to the propulsion plugin

File: hector_quadrotor/hector_quadrotor_controller/urdf/quadrotor_controller.urdf.xacro (robot description, xacro)
@@ -5,27 +5,18 @@
 >
   <!-- Quadrotor Controller Plugin -->
-  <xacro:macro name="quadrotor_controller">
+  <xacro:macro name="quadrotor_controller" params="state_topic imu_topic">
     <gazebo>
-      <controller:hector_quadrotor_pose_estimation name="quadrotor_pose_estimation" plugin="libgazebo_rtt_plugin.so">
-        <import>hector_pose_estimation_rtt</import>
-        <component>hector_pose_estimation::PoseEstimationTaskContext</component>
-        <port name="raw_imu" queue_size="10" />
-        <port name="magnetic" />
-        <port name="pressure_height" />
-        <port name="fix" />
-        <port name="fix_velocity" />
-        <port name="state" queue_size="10" />
-        <port name="imu" queue_size="10" />
-      </controller:hector_quadrotor_pose_estimation>
       <controller:hector_quadrotor_controller name="quadrotor_controller" plugin="libhector_quadrotor_controller.so">
+        <updateRate>100.0</updateRate>
         <import>quadro</import>
         <component>Controller</component>
-        <configuration>$(find hector_quadrotor_controller)/conf/controller.cpf</configuration>
+        <configuration>$(find quadro)/conf/controller.cpf</configuration>
         <port name="sonar_height" />
         <port name="command_velocity" topic="cmd_vel" />
-        <port name="state" queue_size="10" />
-        <port name="imu" queue_size="10" />
+        <port name="state" topic="${state_topic}" queue_size="10" />
+        <port name="imu" topic="${imu_topic}" queue_size="10" />
         <port name="motor_status" />
         <port name="motor_output" topic="motor_pwm" queue_size="10" />
+        <port name="height" />
       </controller:hector_quadrotor_controller>
     </gazebo>

File: hector_quadrotor/hector_quadrotor_controller/urdf/quadrotor_propulsion.urdf.xacro (robot description, xacro)
@@ -11,6 +11,7 @@
         <updateRate>0.0</updateRate>
         <bodyName>base_link</bodyName>
-        <!-- <controlRate>100.0</controlRate> -->
-        <!-- <controlDelay>0.01</controlDelay> -->
+        <controlRate>100.0</controlRate>
+        <!-- <controlTolerance>0.01</controlTolerance> -->
+        <controlDelay>0.01</controlDelay>
       </controller:hector_gazebo_quadrotor_propulsion>
     </gazebo>

Commit message: hector_quadrotor_gazebo: add pose estimation plugin to the quadrotor_plugins.urdf.xacro if available

File: hector_quadrotor/hector_quadrotor_controller/urdf/quadrotor_controller.urdf.xacro (robot description, xacro)
@@ -7,5 +7,5 @@
   <xacro:macro name="quadrotor_controller" params="state_topic imu_topic">
     <gazebo>
-      <controller:hector_quadrotor_controller name="quadrotor_controller" plugin="libhector_quadrotor_controller.so">
+      <controller:hector_quadrotor_controller name="quadrotor_controller" plugin="libgazebo_rtt_plugin.so">
         <updateRate>100.0</updateRate>
         <import>quadro</import>

File: hector_quadrotor/hector_quadrotor_controller/urdf/quadrotor_pose_estimation.urdf.xacro (robot description, xacro)
@@ -4,6 +4,6 @@
 xmlns:xacro="http://ros.org/wiki/xacro"
 >
-  <!-- Quadrotor Controller Plugin -->
-  <xacro:macro name="quadrotor_controller" params="state_topic imu_topic">
+  <!-- Quadrotor Pose Estimation Plugin -->
+  <xacro:macro name="quadrotor_pose_estimation">
     <gazebo>
       <controller:hector_quadrotor_pose_estimation name="quadrotor_pose_estimation" plugin="libgazebo_rtt_plugin.so">
@@ -19,19 +19,4 @@
         <port name="imu" queue_size="10" />
       </controller:hector_quadrotor_pose_estimation>
-      <controller:mbn name="model_based_navigation" plugin="libgazebo_rtt_plugin.so">
-        <updateRate>100.0</updateRate>
-        <import>quadro</import>
-        <component>Simulink</component>
-        <property name="Model">$(find quadro)/simulink/MBN/RTWmodel_QK_SFSVD_ROS.so</property>
-        <port name="raw_imu" queue_size="10" />
-        <port name="magnetic" />
-        <port name="altimeter" />
-        <port name="fix" />
-        <port name="fix_velocity" />
-        <port name="motor_status" />
-        <port name="state" topic="mbn/state" queue_size="10" />
-        <port name="imu" topic="mbn/imu" queue_size="10" />
-        <port name="log" topic="mbn/log" queue_size="10" />
-      </controller:mbn>
     </gazebo>
   </xacro:macro>
