Commit message: [biorob_description] Corrected link lengths till zylinder clamp at last link

File: biorob_common/biorob_description/urdf/biorob_ultra_x4_hp/biorob_ultra_x4_hp_base.urdf.xacro (robot description, xacro)
@@ -10,5 +10,5 @@
   <xacro:property name="j2_length" value=".270"/>
   <xacro:property name="j3_length" value=".270"/>
-  <xacro:property name="j4_length" value=".115"/>
+  <xacro:property name="j4_length" value=".066"/>
   <xacro:property name="pi" value="3.1415926536"/>
   <xacro:macro name="default_inertial" params="mass">

File: biorob_common/biorob_description/urdf/biorob_ultra_x6/biorob_ultra_x6_base.urdf.xacro (robot description, xacro)
@@ -11,6 +11,6 @@
   <xacro:property name="j3_length" value=".10"/>
   <xacro:property name="j4_length" value=".205"/>
-  <xacro:property name="j5_length" value=".14"/>
-  <xacro:property name="j6_length" value=".08"/>
+  <xacro:property name="j5_length" value=".122"/>
+  <xacro:property name="j6_length" value=".045"/>
   <xacro:property name="pi" value="3.1415926536"/>
   <xacro:macro name="default_inertial" params="mass">

File: biorob_common/biorob_description/urdf/biorob_v3_x4/biorob_v3_x4_base.urdf.xacro (robot description, xacro)
@@ -9,6 +9,6 @@
   <!--0.285 to base plate-->
   <xacro:property name="j2_length" value=".307"/>
-  <xacro:property name="j3_length" value=".310"/>
-  <xacro:property name="j4_length" value=".103"/>
+  <xacro:property name="j3_length" value=".311"/>
+  <xacro:property name="j4_length" value=".047"/>
   <xacro:property name="pi" value="3.1415926536"/>
   <xacro:macro name="default_inertial" params="mass">

Commit message: [biorob_description] Corrected link lengths till zylinder clamp at last link / Added description for IK creation of biorob ultra x5_hg and x5_ug

File: biorob_common/biorob_description/urdf/biorob_ultra_x4_hp/biorob_ultra_x4_hp_base.urdf.xacro (robot description, xacro)
@@ -4,5 +4,5 @@
 xmlns:interface="http://playerstage.sourceforge.net/gazebo/xmlschema/#interface"
 xmlns:xacro="http://playerstage.sourceforge.net/gazebo/xmlschema/#interface"
-name="biorob_ultra_x4">
+name="biorob_ultra_x4_hp">
   <xacro:property name="base_height" value=".009"/>
   <xacro:property name="j1_length" value=".284"/>
@@ -19,5 +19,5 @@
     </inertial>
   </xacro:macro>
-  <macro name="biorob_ultra_x4_arm" params="parent *origin">
+  <macro name="biorob_ultra_x4_hp_arm" params="parent *origin">
     <link name="biorob_base_link">
       <visual>

File: biorob_common/biorob_description/urdf/biorob_ultra_x5_hg_as_x4/biorob_ultra_x5_hg_as_x4.urdf.xacro (robot description, xacro)
@@ -1,9 +1,9 @@
 <?xml version="1.0"?>
-<robot name="biorob_ultra_x4_hp"
+<robot name="biorob_ultra_x5_hg_as_x4"
     xmlns:sensor="http://playerstage.sourceforge.net/gazebo/xmlschema/#sensor"
     xmlns:controller="http://playerstage.sourceforge.net/gazebo/xmlschema/#controller"
     xmlns:interface="http://playerstage.sourceforge.net/gazebo/xmlschema/#interface">
     <!-- Included URDF Files -->
-    <include filename="$(find biorob_description)/urdf/biorob_ultra_x4_hp/biorob_ultra_x4_hp_base.urdf.xacro" />
+    <include filename="$(find biorob_description)/urdf/biorob_ultra_x5_hg_as_x4/biorob_ultra_x5_hg_as_x4_base.urdf.xacro" />
     <link name="base">
       <inertial>
@@ -15,6 +15,6 @@
 	</inertial>
       </link>
-    <biorob_ultra_x4_hp_arm parent="base" >
+    <biorob_ultra_x5_hg_as_x4_arm parent="base" >
         <origin xyz="0 0 0" rpy="0 0 0"/>
-    </biorob_ultra_x4_hp_arm>
+    </biorob_ultra_x5_hg_as_x4_arm>
 </robot>

File: biorob_common/biorob_description/urdf/biorob_ultra_x5_hg_as_x4/biorob_ultra_x5_hg_as_x4_base.urdf.xacro (robot description, xacro)
@@ -1,16 +1,14 @@
 <?xml version="1.0"?>
 <robot xmlns:sensor="http://playerstage.sourceforge.net/gazebo/xmlschema/#sensor"
-       xmlns:controller="http://playerstage.sourceforge.net/gazebo/xmlschema/#controller"
-       xmlns:interface="http://playerstage.sourceforge.net/gazebo/xmlschema/#interface"
-       xmlns:xacro="http://playerstage.sourceforge.net/gazebo/xmlschema/#interface"
-       name="biorob_ultra_x5_hg">
-  <xacro:property name="base_height" value=".01"/>
+xmlns:controller="http://playerstage.sourceforge.net/gazebo/xmlschema/#controller"
+xmlns:interface="http://playerstage.sourceforge.net/gazebo/xmlschema/#interface"
+xmlns:xacro="http://playerstage.sourceforge.net/gazebo/xmlschema/#interface"
+name="biorob_ultra_x5_hg_as_x4">
+  <xacro:property name="base_height" value=".009"/>
   <xacro:property name="j1_length" value=".284"/>
   <!--0.285 to base plate-->
   <xacro:property name="j2_length" value=".305"/>
   <xacro:property name="j3_length" value=".305"/>
-  <!--<xacro:property name="j4_length" value=".205"/>-->
-  <xacro:property name="j5_length" value=".122"/>
-  <xacro:property name="j6_length" value=".045"/>
+  <xacro:property name="j4_length" value=".167"/>
   <xacro:property name="pi" value="3.1415926536"/>
   <xacro:macro name="default_inertial" params="mass">
@@ -21,5 +19,5 @@
     </inertial>
   </xacro:macro>
-  <macro name="biorob_ultra_x5_hg_arm" params="parent *origin">
+  <macro name="biorob_ultra_x5_hg_as_x4_arm" params="parent *origin">
     <link name="biorob_base_link">
       <visual>
@@ -122,26 +120,4 @@
       <!--<material>HLUGV/Green</material>-->
     </gazebo>
-  <!--  <link name="biorob_link4">
-      <visual>
-        <geometry>
-          <mesh filename="package://biorob_description/meshes/biorob_x6/biorob_v3_x6_link_4.dae"/>
-        </geometry>
-        <origin xyz="0 0 0" rpy="${pi/2} 0 ${pi/2}"/>
-        <material name="red">
-                </material>
-      </visual>
-      <collision>
-        <geometry>
-          <mesh filename="package://biorob_description/meshes/biorob_x6/biorob_v3_x6_link_4.dae"/>
-        </geometry>
-        <origin xyz="0 0 0" rpy="${pi/2} 0 ${pi/2}"/>
-      </collision>
-      <xacro:default_inertial mass="0.01"/>
-    </link>-->
-    <gazebo reference="biorob_link4">
-      <selfCollide>true</selfCollide>
-      <material>biorob_material/Grey</material>
-      <!--<material>HLUGV/Green</material>-->
-    </gazebo>
     <link name="biorob_link4">
       <visual>
@@ -161,5 +137,5 @@
         <origin xyz="0 0 0" rpy="${pi/2} 0 ${pi/2}"/>
       </collision>
-      <xacro:default_inertial mass="0.01"/>
+      <xacro:default_inertial mass="0.1"/>
     </link>
     <gazebo reference="biorob_link4">
@@ -168,28 +144,4 @@
       <!--<material>HLUGV/Green</material>-->
     </gazebo>
-    <link name="biorob_link5">
-      <visual>
-        <geometry>
-          <mesh filename="package://biorob_description/meshes/biorob_ultra/biorob_ultra_tcp_end_80.dae"/>
-          <!--<cylinder radius="0.002" length="0.001" />-->
-        </geometry>
-        <origin xyz="0 0 0" rpy="0 0 0"/>
-        <material name="red">
-                </material>
-      </visual>
-      <collision>
-        <geometry>
-          <mesh filename="package://biorob_description/meshes/biorob_ultra/biorob_ultra_tcp_end_80.dae"/>
-          <!--<cylinder radius="0.002" length="0.001" />-->
-        </geometry>
-        <origin xyz="0 0 0" rpy="0 0 0"/>
-      </collision>
-      <xacro:default_inertial mass="0.01"/>
-    </link>
-    <gazebo reference="biorob_link5">
-      <selfCollide>true</selfCollide>
-      <material>biorob_material/Grey</material>
-      <!--<material>HLUGV/Green</material>-->
-    </gazebo>
     <link name="biorob_toolframe">
       <visual>
@@ -197,13 +149,13 @@
           <cylinder radius="0.01" length="0.001" />
         </geometry>
-        <origin xyz="0 0 0" rpy="0 0 0"/>
-        <material name="red">
-        </material>
-      </visual>
-      <collision>
-        <geometry>
-          <cylinder radius="0.01" length="0.001" />
-        </geometry>
-        <origin xyz="0 0 0" rpy="0 0 0"/>
+        <origin xyz="0 0 0" rpy="${pi/2} 0 ${pi/2}"/>
+        <material name="red">
+        </material>
+      </visual>
+      <collision>
+        <geometry>
+          <cylinder radius="0.02" length="0.001" />
+        </geometry>
+        <origin xyz="0 0 0" rpy="${pi/2} 0 ${pi/2}"/>
       </collision>
       <xacro:default_inertial mass="0.05"/>
@@ -243,31 +195,14 @@
       <child link="biorob_link4"/>
       <axis xyz="0 0 1"/>
-      <origin xyz="${j3_length} 0 0"/>
+      <origin xyz="${j3_length} 0 0.0"/>
       <limit effort="6.0" lower="${-pi*(100/180)}" upper="${pi*(100/180)}" velocity="1.5708"/>
       <!-- TODO: give correct effort limits -->
       <dynamics damping="1.0" friction="1.0"/>
     </joint>
-<!--    <joint name="joint5" type="revolute">
+    <joint name="tool_frame" type="fixed">
       <parent link="biorob_link4"/>
-      <child link="biorob_link5"/>
-      <axis xyz="0 0 1"/>
-      <origin xyz="${j4_length} 0 0.0"/>
-      <limit effort="6.0" lower="${-pi*(100/180)}" upper="${pi*(100/180)}" velocity="1.5708"/>
-      <dynamics damping="1.0" friction="1.0"/>
-    </joint>-->
-    <joint name="joint5" type="revolute">
-      <parent link="biorob_link4"/>
-      <child link="biorob_link5"/>
-      <axis xyz="0 0 1"/>
-      <origin xyz="${j5_length} 0 0" rpy="${pi/2} 0 ${pi/2}"/>
-      <limit effort="6.0" lower="${-pi*(100/180)}" upper="${pi*(100/180)}" velocity="1.5708"/>
-      <!-- TODO: give correct effort limits -->
-      <dynamics damping="1.0" friction="1.0"/>
-    </joint>
-    <joint name="tool_frame" type="fixed">
-      <parent link="biorob_link5"/>
       <child link="biorob_toolframe"/>
       <axis xyz="0 0 1"/>
-      <origin xyz="0 0 ${j6_length}" rpy="0 0 0"/>
+      <origin xyz="${j4_length} 0.0 0.0" rpy="0 0 0"/>
     </joint>
     <transmission type="pr2_mechanism_model/SimpleTransmission" name="joint1_trans">
@@ -291,15 +226,5 @@
       <mechanicalReduction>1.0</mechanicalReduction>
     </transmission>
-    <transmission type="pr2_mechanism_model/SimpleTransmission" name="joint5_trans">
-      <actuator name="joint5_motor"/>
-      <joint name="joint5"/>
-      <mechanicalReduction>1.0</mechanicalReduction>
-    </transmission>
-    <transmission type="pr2_mechanism_model/SimpleTransmission" name="joint6_trans">
-      <actuator name="joint6_motor"/>
-      <joint name="joint6"/>
-      <mechanicalReduction>1.0</mechanicalReduction>
-    </transmission>
-    <!--    <gazebo reference="biorob_toolframe">
+<!--    <gazebo reference="biorob_toolframe">
       <sensor:camera name="finger_tip_camera_sensor">
         <imageSize>640 480</imageSize>
@@ -314,17 +239,17 @@
           <imageTopicName>finger_tip_cam/image</imageTopicName>
           <frameName>biorob_toolframe</frameName>
-          <interface:camera name="finger_tip_camera_iface" />
+          <interface:camera name="finger_tip_camera_iface"/>
         </controller:gazebo_ros_camera>
       </sensor:camera>
       <turnGravityOff>true</turnGravityOff>
       <material>PR2/Blue</material>
+    </gazebo>
+    <gazebo>
+      <controller:gazebo_ros_controller_manager name="gazebo_ros_controller_manager" plugin="libgazebo_ros_controller_manager.so">
+        <alwaysOn>true</alwaysOn>
+        <updateRate>100.0</updateRate>
+        <interface:audio name="gazebo_ros_controller_manager_dummy_iface_biorob"/>
+      </controller:gazebo_ros_controller_manager>
     </gazebo>-->
-    <!--        <gazebo>
-              <controller:gazebo_ros_controller_manager name="gazebo_ros_controller_manager" plugin="libgazebo_ros_controller_manager.so">
-                <alwaysOn>true</alwaysOn>
-                <updateRate>100.0</updateRate>
-                <interface:audio name="gazebo_ros_controller_manager_dummy_iface_biorob" />
-              </controller:gazebo_ros_controller_manager>
-            </gazebo>-->
   </macro>
 </robot>

File: biorob_common/biorob_description/urdf/biorob_ultra_x5_ug/biorob_ultra_x5_ug_base.urdf.xacro (robot description, xacro)
@@ -11,5 +11,5 @@
   <xacro:property name="j3_length" value=".100"/>
   <xacro:property name="j4_length" value=".205"/>
-  <xacro:property name="j5_length" value=".150"/>
+  <xacro:property name="j5_length" value=".066"/>
   <!--<xacro:property name="j6_length" value=".08"/>-->
   <xacro:property name="pi" value="3.1415926536"/>

File: biorob_common/biorob_description/urdf/biorob_ultra_x5_ug_as_x6/biorob_ultra_x5_ug_as_x6.urdf.xacro (robot description, xacro)
@@ -1,9 +1,9 @@
 <?xml version="1.0"?>
-<robot name="biorob_ultra_x4_hp"
+<robot name="biorob_ultra_x5_ug_as_x6"
     xmlns:sensor="http://playerstage.sourceforge.net/gazebo/xmlschema/#sensor"
     xmlns:controller="http://playerstage.sourceforge.net/gazebo/xmlschema/#controller"
     xmlns:interface="http://playerstage.sourceforge.net/gazebo/xmlschema/#interface">
     <!-- Included URDF Files -->
-    <include filename="$(find biorob_description)/urdf/biorob_ultra_x4_hp/biorob_ultra_x4_hp_base.urdf.xacro" />
+    <include filename="$(find biorob_description)/urdf/biorob_ultra_x5_ug_as_x6/biorob_ultra_x5_ug_as_x6_base.urdf.xacro" />
     <link name="base">
       <inertial>
@@ -15,6 +15,6 @@
 	</inertial>
       </link>
-    <biorob_ultra_x4_hp_arm parent="base" >
+    <biorob_ultra_x5_ug_as_x6_arm parent="base" >
         <origin xyz="0 0 0" rpy="0 0 0"/>
-    </biorob_ultra_x4_hp_arm>
+    </biorob_ultra_x5_ug_as_x6_arm>
 </robot>

File: biorob_common/biorob_description/urdf/biorob_ultra_x5_ug_as_x6/biorob_ultra_x5_ug_as_x6_base.urdf.xacro (robot description, xacro)
@@ -4,13 +4,13 @@
        xmlns:interface="http://playerstage.sourceforge.net/gazebo/xmlschema/#interface"
        xmlns:xacro="http://playerstage.sourceforge.net/gazebo/xmlschema/#interface"
-       name="biorob_ultra_x5_hg">
+       name="biorob_ultra_x5_ug_as_x6">
   <xacro:property name="base_height" value=".01"/>
   <xacro:property name="j1_length" value=".284"/>
   <!--0.285 to base plate-->
   <xacro:property name="j2_length" value=".305"/>
-  <xacro:property name="j3_length" value=".305"/>
-  <!--<xacro:property name="j4_length" value=".205"/>-->
-  <xacro:property name="j5_length" value=".122"/>
-  <xacro:property name="j6_length" value=".045"/>
+  <xacro:property name="j3_length" value=".10"/>
+  <xacro:property name="j4_length" value=".205"/>
+  <xacro:property name="j5_length" value=".066"/>
+  <xacro:property name="j6_length" value=".0"/>
   <xacro:property name="pi" value="3.1415926536"/>
   <xacro:macro name="default_inertial" params="mass">
@@ -21,5 +21,5 @@
     </inertial>
   </xacro:macro>
-  <macro name="biorob_ultra_x5_hg_arm" params="parent *origin">
+  <macro name="biorob_ultra_x5_ug_as_x6_arm" params="parent *origin">
     <link name="biorob_base_link">
       <visual>
@@ -101,5 +101,5 @@
       <visual>
         <geometry>
-          <mesh filename="package://biorob_description/meshes/biorob_common/biorob_link_3.dae"/>
+          <mesh filename="package://biorob_description/meshes/biorob_x6/biorob_v3_x6_link_3.dae"/>
           <!--<cylinder radius="0.02" length="${j3_length}" />-->
         </geometry>
@@ -110,5 +110,5 @@
       <collision>
         <geometry>
-          <mesh filename="package://biorob_description/meshes/biorob_common/biorob_link_3.dae"/>
+          <mesh filename="package://biorob_description/meshes/biorob_x6/biorob_v3_x6_link_3.dae"/>
           <!--  <cylinder radius="0.02" length="${j3_length}" />-->
         </geometry>
@@ -122,10 +122,11 @@
       <!--<material>HLUGV/Green</material>-->
     </gazebo>
-  <!--  <link name="biorob_link4">
+    <link name="biorob_link4">
       <visual>
         <geometry>
           <mesh filename="package://biorob_description/meshes/biorob_x6/biorob_v3_x6_link_4.dae"/>
-        </geometry>
-        <origin xyz="0 0 0" rpy="${pi/2} 0 ${pi/2}"/>
+          <!--                    <cylinder radius="0.002" length="0.001" />-->
+        </geometry>
+        <origin xyz="0 0 0" rpy="0 0 0"/>
         <material name="red">
                 </material>
@@ -134,15 +135,16 @@
         <geometry>
           <mesh filename="package://biorob_description/meshes/biorob_x6/biorob_v3_x6_link_4.dae"/>
-        </geometry>
-        <origin xyz="0 0 0" rpy="${pi/2} 0 ${pi/2}"/>
+          <!--<cylinder radius="0.02" length="${j4_length}" />-->
+        </geometry>
+        <origin xyz="0 0 0" rpy="0 0 0"/>
       </collision>
       <xacro:default_inertial mass="0.01"/>
-    </link>-->
-    <gazebo reference="biorob_link4">
-      <selfCollide>true</selfCollide>
-      <material>biorob_material/Grey</material>
-      <!--<material>HLUGV/Green</material>-->
-    </gazebo>
-    <link name="biorob_link4">
+    </link>
+    <gazebo reference="biorob_link5">
+      <selfCollide>true</selfCollide>
+      <material>biorob_material/Grey</material>
+      <!--<material>HLUGV/Green</material>-->
+    </gazebo>
+    <link name="biorob_link5">
       <visual>
         <geometry>
@@ -150,5 +152,5 @@
           <!--  <cylinder radius="0.02" length="${j4_length}" />-->
         </geometry>
-        <origin xyz="0 0 0" rpy="${pi/2} 0 ${pi/2}"/>
+        <origin xyz="0 0 0" rpy="${pi/2} 0 0"/>
         <material name="red">
                 </material>
@@ -159,14 +161,14 @@
           <!--<cylinder radius="0.02" length="${j4_length}" />-->
         </geometry>
-        <origin xyz="0 0 0" rpy="${pi/2} 0 ${pi/2}"/>
+        <origin xyz="0 0 0" rpy="${pi/2} 0 0"/>
       </collision>
       <xacro:default_inertial mass="0.01"/>
     </link>
-    <gazebo reference="biorob_link4">
-      <selfCollide>true</selfCollide>
-      <material>biorob_material/Grey</material>
-      <!--<material>HLUGV/Green</material>-->
-    </gazebo>
-    <link name="biorob_link5">
+    <gazebo reference="biorob_link5">
+      <selfCollide>true</selfCollide>
+      <material>biorob_material/Grey</material>
+      <!--<material>HLUGV/Green</material>-->
+    </gazebo>
+    <link name="biorob_link6">
       <visual>
         <geometry>
@@ -187,5 +189,5 @@
       <xacro:default_inertial mass="0.01"/>
     </link>
-    <gazebo reference="biorob_link5">
+    <gazebo reference="biorob_link6">
       <selfCollide>true</selfCollide>
       <material>biorob_material/Grey</material>
@@ -203,5 +205,5 @@
       <collision>
         <geometry>
-          <cylinder radius="0.01" length="0.001" />
+          <cylinder radius="0.02" length="0.001" />
         </geometry>
         <origin xyz="0 0 0" rpy="0 0 0"/>
@@ -243,28 +245,29 @@
       <child link="biorob_link4"/>
       <axis xyz="0 0 1"/>
-      <origin xyz="${j3_length} 0 0"/>
+      <origin xyz="${j3_length} 0 0.0" rpy="${pi/2} 0 ${pi/2}"/>
       <limit effort="6.0" lower="${-pi*(100/180)}" upper="${pi*(100/180)}" velocity="1.5708"/>
       <!-- TODO: give correct effort limits -->
       <dynamics damping="1.0" friction="1.0"/>
     </joint>
-<!--    <joint name="joint5" type="revolute">
-      <parent link="biorob_link4"/>
-      <child link="biorob_link5"/>
-      <axis xyz="0 0 1"/>
-      <origin xyz="${j4_length} 0 0.0"/>
-      <limit effort="6.0" lower="${-pi*(100/180)}" upper="${pi*(100/180)}" velocity="1.5708"/>
-      <dynamics damping="1.0" friction="1.0"/>
-    </joint>-->
     <joint name="joint5" type="revolute">
       <parent link="biorob_link4"/>
       <child link="biorob_link5"/>
       <axis xyz="0 0 1"/>
-      <origin xyz="${j5_length} 0 0" rpy="${pi/2} 0 ${pi/2}"/>
+      <origin xyz="0 0 ${j4_length}" rpy="${-pi/2} 0 0"/>
       <limit effort="6.0" lower="${-pi*(100/180)}" upper="${pi*(100/180)}" velocity="1.5708"/>
       <!-- TODO: give correct effort limits -->
       <dynamics damping="1.0" friction="1.0"/>
     </joint>
+    <joint name="joint6" type="revolute">
+      <parent link="biorob_link5"/>
+      <child link="biorob_link6"/>
+      <axis xyz="0 0 1"/>
+      <origin xyz="0 ${-j5_length} 0 " rpy="${pi/2} 0 0"/>
+      <limit effort="6.0" lower="${-pi*(100/180)}" upper="${pi*(100/180)}" velocity="1.5708"/>
+      <!-- TODO: give correct effort limits -->
+      <dynamics damping="1.0" friction="1.0"/>
+    </joint>
     <joint name="tool_frame" type="fixed">
-      <parent link="biorob_link5"/>
+      <parent link="biorob_link6"/>
       <child link="biorob_toolframe"/>
       <axis xyz="0 0 1"/>

File: biorob_common/biorob_description/urdf/biorob_v3_x6/biorob_v3_x6_base.urdf.xacro (robot description, xacro)
@@ -9,8 +9,8 @@
   <!--0.285 to base plate-->
   <xacro:property name="j2_length" value=".307"/>
-  <xacro:property name="j3_length" value=".10"/>
-  <xacro:property name="j4_length" value=".209"/>
-  <xacro:property name="j5_length" value=".103"/>
-  <xacro:property name="j6_length" value=".021"/>
+  <xacro:property name="j3_length" value=".10" comment=".130"/>
+  <xacro:property name="j4_length" value=".209" comment=".181"/>
+  <xacro:property name="j5_length" value=".103" comment=".122"/>
+  <xacro:property name="j6_length" value=".021" comment=".018 rohr zu rohr / .012 rot achse zu Befestigung .012"/>
   <xacro:property name="pi" value="3.1415926536"/>
   <xacro:macro name="default_inertial" params="mass">
