Commit message: [biorob_description] Corrected link lengths till zylinder clamp at last link

File: biorob_common/biorob_description/urdf/biorob_ultra_x4/biorob_ultra_x4_base.urdf.xacro (robot description, xacro)
@@ -10,5 +10,5 @@
   <xacro:property name="j2_length" value=".305"/>
   <xacro:property name="j3_length" value=".305"/>
-  <xacro:property name="j4_length" value=".150"/>
+  <xacro:property name="j4_length" value=".066"/>
   <xacro:property name="pi" value="3.1415926536"/>
   <xacro:macro name="default_inertial" params="mass">

Commit message: [biorob_description] Corrected link lengths till zylinder clamp at last link / Added description for IK creation of biorob ultra x5_hg and x5_ug

File: biorob_common/biorob_description/urdf/biorob_ultra_x4/biorob_ultra_x4_base.urdf.xacro (robot description, xacro)
@@ -5,6 +5,6 @@
 xmlns:xacro="http://playerstage.sourceforge.net/gazebo/xmlschema/#interface"
 name="biorob_ultra_x4">
-  <xacro:property name="base_height" value=".009"/>
-  <xacro:property name="j1_length" value=".284"/>
+  <xacro:property name="base_height" value=".008"/>
+  <xacro:property name="j1_length" value=".277"/>
   <!--0.285 to base plate-->
   <xacro:property name="j2_length" value=".305"/>

File: biorob_common/biorob_description/urdf/biorob_ultra_x4_hp/biorob_ultra_x4_hp_base.urdf.xacro (robot description, xacro)
@@ -5,6 +5,6 @@
 xmlns:xacro="http://playerstage.sourceforge.net/gazebo/xmlschema/#interface"
 name="biorob_ultra_x4_hp">
-  <xacro:property name="base_height" value=".009"/>
-  <xacro:property name="j1_length" value=".284"/>
+  <xacro:property name="base_height" value=".008"/>
+  <xacro:property name="j1_length" value=".277"/>
   <!--0.285 to base plate-->
   <xacro:property name="j2_length" value=".270"/>

File: biorob_common/biorob_description/urdf/biorob_ultra_x5_hg/biorob_ultra_x5_hg_base.urdf.xacro (robot description, xacro)
@@ -5,6 +5,6 @@
        xmlns:xacro="http://playerstage.sourceforge.net/gazebo/xmlschema/#interface"
        name="biorob_ultra_x5_hg">
-  <xacro:property name="base_height" value=".01"/>
-  <xacro:property name="j1_length" value=".284"/>
+  <xacro:property name="base_height" value=".008"/>
+  <xacro:property name="j1_length" value=".277"/>
   <!--0.285 to base plate-->
   <xacro:property name="j2_length" value=".305"/>

File: biorob_common/biorob_description/urdf/biorob_ultra_x5_hg_as_x4/biorob_ultra_x5_hg_as_x4_base.urdf.xacro (robot description, xacro)
@@ -5,6 +5,6 @@
 xmlns:xacro="http://playerstage.sourceforge.net/gazebo/xmlschema/#interface"
 name="biorob_ultra_x5_hg_as_x4">
-  <xacro:property name="base_height" value=".009"/>
-  <xacro:property name="j1_length" value=".284"/>
+  <xacro:property name="base_height" value=".008"/>
+  <xacro:property name="j1_length" value=".277"/>
   <!--0.285 to base plate-->
   <xacro:property name="j2_length" value=".305"/>

File: biorob_common/biorob_description/urdf/biorob_ultra_x5_ug/biorob_ultra_x5_ug_base.urdf.xacro (robot description, xacro)
@@ -5,6 +5,6 @@
        xmlns:xacro="http://playerstage.sourceforge.net/gazebo/xmlschema/#interface"
        name="biorob_ultra_x5_ug">
-  <xacro:property name="base_height" value=".01"/>
-  <xacro:property name="j1_length" value=".284"/>
+  <xacro:property name="base_height" value=".008"/>
+  <xacro:property name="j1_length" value=".277"/>
   <!--0.285 to base plate-->
   <xacro:property name="j2_length" value=".305"/>

File: biorob_common/biorob_description/urdf/biorob_ultra_x5_ug_as_x6/biorob_ultra_x5_ug_as_x6_base.urdf.xacro (robot description, xacro)
@@ -5,9 +5,9 @@
        xmlns:xacro="http://playerstage.sourceforge.net/gazebo/xmlschema/#interface"
        name="biorob_ultra_x5_ug_as_x6">
-  <xacro:property name="base_height" value=".01"/>
-  <xacro:property name="j1_length" value=".284"/>
+  <xacro:property name="base_height" value=".008"/>
+  <xacro:property name="j1_length" value=".277"/>
   <!--0.285 to base plate-->
   <xacro:property name="j2_length" value=".305"/>
-  <xacro:property name="j3_length" value=".10"/>
+  <xacro:property name="j3_length" value=".100"/>
   <xacro:property name="j4_length" value=".205"/>
   <xacro:property name="j5_length" value=".066"/>

File: biorob_common/biorob_description/urdf/biorob_ultra_x6/biorob_ultra_x6_base.urdf.xacro (robot description, xacro)
@@ -5,6 +5,6 @@
        xmlns:xacro="http://playerstage.sourceforge.net/gazebo/xmlschema/#interface"
        name="biorob_ultra_x6">
-  <xacro:property name="base_height" value=".01"/>
-  <xacro:property name="j1_length" value=".284"/>
+  <xacro:property name="base_height" value=".008"/>
+  <xacro:property name="j1_length" value=".277"/>
   <!--0.285 to base plate-->
   <xacro:property name="j2_length" value=".305"/>

File: biorob_common/biorob_description/urdf/biorob_v3_x4/biorob_v3_x4_base.urdf.xacro (robot description, xacro)
@@ -5,6 +5,6 @@
 xmlns:xacro="http://playerstage.sourceforge.net/gazebo/xmlschema/#interface"
 name="biorob_v3_x4">
-  <xacro:property name="base_height" value=".009"/>
-  <xacro:property name="j1_length" value=".276"/>
+  <xacro:property name="base_height" value=".008"/>
+  <xacro:property name="j1_length" value=".277"/>
   <!--0.285 to base plate-->
   <xacro:property name="j2_length" value=".307"/>

File: biorob_common/biorob_description/urdf/biorob_v3_x6/biorob_v3_x6_base.urdf.xacro (robot description, xacro)
@@ -5,12 +5,12 @@
        xmlns:xacro="http://playerstage.sourceforge.net/gazebo/xmlschema/#interface"
        name="biorob_v3_x6">
-  <xacro:property name="base_height" value=".009"/>
-  <xacro:property name="j1_length" value=".276"/>
+  <xacro:property name="base_height" value=".008"/>
+  <xacro:property name="j1_length" value=".277"/>
   <!--0.285 to base plate-->
   <xacro:property name="j2_length" value=".307"/>
-  <xacro:property name="j3_length" value=".10" comment=".130"/>
-  <xacro:property name="j4_length" value=".209" comment=".181"/>
-  <xacro:property name="j5_length" value=".103" comment=".122"/>
-  <xacro:property name="j6_length" value=".021" comment=".018 rohr zu rohr / .012 rot achse zu Befestigung .012"/>
+  <xacro:property name="j3_length" value=".130"/>
+  <xacro:property name="j4_length" value=".181"/>
+  <xacro:property name="j5_length" value=".126"/>
+  <xacro:property name="j6_length" value=".018"/>
   <xacro:property name="pi" value="3.1415926536"/>
   <xacro:macro name="default_inertial" params="mass">

Commit message: [biorob_description] Updated base length and usage in origin determination of joint 2

File: biorob_common/biorob_description/urdf/biorob_ultra_x4/biorob_ultra_x4_base.urdf.xacro (robot description, xacro)
@@ -6,6 +6,6 @@
 name="biorob_ultra_x4">
   <xacro:property name="base_height" value=".008"/>
-  <xacro:property name="j1_length" value=".277"/>
-  <!--0.285 to base plate-->
+  <xacro:property name="j1_length" value=".276"/>
+  <!--0.284 to base plate-->
   <xacro:property name="j2_length" value=".305"/>
   <xacro:property name="j3_length" value=".305"/>
@@ -179,5 +179,5 @@
       <child link="biorob_link2"/>
       <axis xyz="0 0 1"/>
-      <origin xyz="0 0 ${j1_length-base_height}" rpy="${pi/2} 0 0"/>
+      <origin xyz="0 0 ${j1_length}" rpy="${pi/2} 0 0"/>
       <limit effort="6.0" lower="${-pi*(170/180)}" upper="${pi*(170/180)}" velocity="1.5708"/>
       <dynamics damping="1.0" friction="1.0"/>

File: biorob_common/biorob_description/urdf/biorob_ultra_x4_hp/biorob_ultra_x4_hp_base.urdf.xacro (robot description, xacro)
@@ -6,6 +6,6 @@
 name="biorob_ultra_x4_hp">
   <xacro:property name="base_height" value=".008"/>
-  <xacro:property name="j1_length" value=".277"/>
-  <!--0.285 to base plate-->
+  <xacro:property name="j1_length" value=".276"/>
+  <!--0.284 to base plate-->
   <xacro:property name="j2_length" value=".270"/>
   <xacro:property name="j3_length" value=".270"/>
@@ -179,5 +179,5 @@
       <child link="biorob_link2"/>
       <axis xyz="0 0 1"/>
-      <origin xyz="0 0 ${j1_length-base_height}" rpy="${pi/2} 0 0"/>
+      <origin xyz="0 0 ${j1_length}" rpy="${pi/2} 0 0"/>
       <limit effort="6.0" lower="${-pi*(170/180)}" upper="${pi*(170/180)}" velocity="1.5708"/>
       <dynamics damping="1.0" friction="1.0"/>

File: biorob_common/biorob_description/urdf/biorob_ultra_x5_hg/biorob_ultra_x5_hg_base.urdf.xacro (robot description, xacro)
@@ -6,6 +6,6 @@
        name="biorob_ultra_x5_hg">
   <xacro:property name="base_height" value=".008"/>
-  <xacro:property name="j1_length" value=".277"/>
-  <!--0.285 to base plate-->
+  <xacro:property name="j1_length" value=".276"/>
+  <!--0.284 to base plate-->
   <xacro:property name="j2_length" value=".305"/>
   <xacro:property name="j3_length" value=".305"/>
@@ -227,5 +227,5 @@
       <child link="biorob_link2"/>
       <axis xyz="0 0 1"/>
-      <origin xyz="0 0 ${j1_length-base_height}" rpy="${pi/2} 0 0"/>
+      <origin xyz="0 0 ${j1_length}" rpy="${pi/2} 0 0"/>
       <limit effort="6.0" lower="${-pi*(170/180)}" upper="${pi*(170/180)}" velocity="1.5708"/>
       <dynamics damping="1.0" friction="1.0"/>

File: biorob_common/biorob_description/urdf/biorob_ultra_x5_hg_as_x4/biorob_ultra_x5_hg_as_x4_base.urdf.xacro (robot description, xacro)
@@ -6,6 +6,6 @@
 name="biorob_ultra_x5_hg_as_x4">
   <xacro:property name="base_height" value=".008"/>
-  <xacro:property name="j1_length" value=".277"/>
-  <!--0.285 to base plate-->
+  <xacro:property name="j1_length" value=".276"/>
+  <!--0.284 to base plate-->
   <xacro:property name="j2_length" value=".305"/>
   <xacro:property name="j3_length" value=".305"/>
@@ -179,5 +179,5 @@
       <child link="biorob_link2"/>
       <axis xyz="0 0 1"/>
-      <origin xyz="0 0 ${j1_length-base_height}" rpy="${pi/2} 0 0"/>
+      <origin xyz="0 0 ${j1_length}" rpy="${pi/2} 0 0"/>
       <limit effort="6.0" lower="${-pi*(170/180)}" upper="${pi*(170/180)}" velocity="1.5708"/>
       <dynamics damping="1.0" friction="1.0"/>

File: biorob_common/biorob_description/urdf/biorob_ultra_x5_ug/biorob_ultra_x5_ug_base.urdf.xacro (robot description, xacro)
@@ -6,6 +6,6 @@
        name="biorob_ultra_x5_ug">
   <xacro:property name="base_height" value=".008"/>
-  <xacro:property name="j1_length" value=".277"/>
-  <!--0.285 to base plate-->
+  <xacro:property name="j1_length" value=".276"/>
+  <!--0.284 to base plate-->
   <xacro:property name="j2_length" value=".305"/>
   <xacro:property name="j3_length" value=".100"/>
@@ -205,5 +205,5 @@
       <child link="biorob_link2"/>
       <axis xyz="0 0 1"/>
-      <origin xyz="0 0 ${j1_length-base_height}" rpy="${pi/2} 0 0"/>
+      <origin xyz="0 0 ${j1_length}" rpy="${pi/2} 0 0"/>
       <limit effort="6.0" lower="${-pi*(170/180)}" upper="${pi*(170/180)}" velocity="1.5708"/>
       <dynamics damping="1.0" friction="1.0"/>

File: biorob_common/biorob_description/urdf/biorob_ultra_x5_ug_as_x6/biorob_ultra_x5_ug_as_x6_base.urdf.xacro (robot description, xacro)
@@ -6,6 +6,6 @@
        name="biorob_ultra_x5_ug_as_x6">
   <xacro:property name="base_height" value=".008"/>
-  <xacro:property name="j1_length" value=".277"/>
-  <!--0.285 to base plate-->
+  <xacro:property name="j1_length" value=".276"/>
+  <!--0.284 to base plate-->
   <xacro:property name="j2_length" value=".305"/>
   <xacro:property name="j3_length" value=".100"/>
@@ -229,5 +229,5 @@
       <child link="biorob_link2"/>
       <axis xyz="0 0 1"/>
-      <origin xyz="0 0 ${j1_length-base_height}" rpy="${pi/2} 0 0"/>
+      <origin xyz="0 0 ${j1_length}" rpy="${pi/2} 0 0"/>
       <limit effort="6.0" lower="${-pi*(170/180)}" upper="${pi*(170/180)}" velocity="1.5708"/>
       <dynamics damping="1.0" friction="1.0"/>

File: biorob_common/biorob_description/urdf/biorob_ultra_x6/biorob_ultra_x6_base.urdf.xacro (robot description, xacro)
@@ -6,8 +6,8 @@
        name="biorob_ultra_x6">
   <xacro:property name="base_height" value=".008"/>
-  <xacro:property name="j1_length" value=".277"/>
-  <!--0.285 to base plate-->
+  <xacro:property name="j1_length" value=".276"/>
+  <!--0.284 to base plate-->
   <xacro:property name="j2_length" value=".305"/>
-  <xacro:property name="j3_length" value=".10"/>
+  <xacro:property name="j3_length" value=".100"/>
   <xacro:property name="j4_length" value=".205"/>
   <xacro:property name="j5_length" value=".122"/>
@@ -229,5 +229,5 @@
       <child link="biorob_link2"/>
       <axis xyz="0 0 1"/>
-      <origin xyz="0 0 ${j1_length-base_height}" rpy="${pi/2} 0 0"/>
+      <origin xyz="0 0 ${j1_length}" rpy="${pi/2} 0 0"/>
       <limit effort="6.0" lower="${-pi*(170/180)}" upper="${pi*(170/180)}" velocity="1.5708"/>
       <dynamics damping="1.0" friction="1.0"/>

File: biorob_common/biorob_description/urdf/biorob_v3_x4/biorob_v3_x4_base.urdf.xacro (robot description, xacro)
@@ -6,6 +6,6 @@
 name="biorob_v3_x4">
   <xacro:property name="base_height" value=".008"/>
-  <xacro:property name="j1_length" value=".277"/>
-  <!--0.285 to base plate-->
+  <xacro:property name="j1_length" value=".276"/>
+  <!--0.284 to base plate-->
   <xacro:property name="j2_length" value=".307"/>
   <xacro:property name="j3_length" value=".311"/>
@@ -179,5 +179,5 @@
       <child link="biorob_link2"/>
       <axis xyz="0 0 1"/>
-      <origin xyz="0 0 ${j1_length-base_height}" rpy="${pi/2} 0 0"/>
+      <origin xyz="0 0 ${j1_length}" rpy="${pi/2} 0 0"/>
       <limit effort="6.0" lower="${-pi*(170/180)}" upper="${pi*(170/180)}" velocity="1.5708"/>
       <dynamics damping="1.0" friction="1.0"/>

File: biorob_common/biorob_description/urdf/biorob_v3_x6/biorob_v3_x6_base.urdf.xacro (robot description, xacro)
@@ -6,6 +6,6 @@
        name="biorob_v3_x6">
   <xacro:property name="base_height" value=".008"/>
-  <xacro:property name="j1_length" value=".277"/>
-  <!--0.285 to base plate-->
+  <xacro:property name="j1_length" value=".276"/>
+  <!--0.284 to base plate-->
   <xacro:property name="j2_length" value=".307"/>
   <xacro:property name="j3_length" value=".130"/>
@@ -215,5 +215,5 @@
       <child link="biorob_link2"/>
       <axis xyz="0 0 1"/>
-      <origin xyz="0 0 ${j1_length-base_height}" rpy="${pi/2} -${pi/2} 0"/>
+      <origin xyz="0 0 ${j1_length}" rpy="${pi/2} -${pi/2} 0"/>
       <limit effort="6.0" lower="${-pi*(170/180)}" upper="${pi*(170/180)}" velocity="1.5708"/>
       <dynamics damping="1.0" friction="1.0"/>
