Commit message: [biorob_description] Updated meshes and fixed wrong links lengths

File: biorob_common/biorob_description/urdf/biorob_ultra_x4/biorob_ultra_x4_base.urdf.xacro (robot description, xacro)
@@ -123,5 +123,5 @@
       <visual>
         <geometry>
-          <mesh filename="package://biorob_description/meshes/biorob_common/biorob_link_4.dae"/>
+          <mesh filename="package://biorob_description/meshes/biorob_common/biorob_link_4_0066.stl"/>
           <!--  <cylinder radius="0.02" length="${j4_length}" />-->
         </geometry>
@@ -132,5 +132,5 @@
       <collision>
         <geometry>
-          <mesh filename="package://biorob_description/meshes/biorob_common/biorob_link_4.dae"/>
+          <mesh filename="package://biorob_description/meshes/biorob_common/biorob_link_4_0066.stl"/>
           <!--<cylinder radius="0.02" length="${j4_length}" />-->
         </geometry>

File: biorob_common/biorob_description/urdf/biorob_ultra_x5_hg/biorob_ultra_x5_hg_base.urdf.xacro (robot description, xacro)
@@ -147,5 +147,5 @@
       <visual>
         <geometry>
-          <mesh filename="package://biorob_description/meshes/biorob_common/biorob_link_4.dae"/>
+          <mesh filename="package://biorob_description/meshes/biorob_common/biorob_link_4_0122.stl"/>
           <!--  <cylinder radius="0.02" length="${j4_length}" />-->
         </geometry>
@@ -156,5 +156,5 @@
       <collision>
         <geometry>
-          <mesh filename="package://biorob_description/meshes/biorob_common/biorob_link_4.dae"/>
+          <mesh filename="package://biorob_description/meshes/biorob_common/biorob_link_4_0122.stl"/>
           <!--<cylinder radius="0.02" length="${j4_length}" />-->
         </geometry>
@@ -171,5 +171,5 @@
       <visual>
         <geometry>
-          <mesh filename="package://biorob_description/meshes/biorob_ultra/biorob_ultra_tcp_end_80.dae"/>
+          <mesh filename="package://biorob_description/meshes/biorob_ultra/biorob_ultra_tcp_end_45.stl"/>
           <!--<cylinder radius="0.002" length="0.001" />-->
         </geometry>
@@ -180,5 +180,5 @@
       <collision>
         <geometry>
-          <mesh filename="package://biorob_description/meshes/biorob_ultra/biorob_ultra_tcp_end_80.dae"/>
+          <mesh filename="package://biorob_description/meshes/biorob_ultra/biorob_ultra_tcp_end_45.stl"/>
           <!--<cylinder radius="0.002" length="0.001" />-->
         </geometry>

File: biorob_common/biorob_description/urdf/biorob_ultra_x6/biorob_ultra_x6_base.urdf.xacro (robot description, xacro)
@@ -149,5 +149,5 @@
       <visual>
         <geometry>
-          <mesh filename="package://biorob_description/meshes/biorob_common/biorob_link_4.dae"/>
+          <mesh filename="package://biorob_description/meshes/biorob_common/biorob_link_4_0122.stl"/>
           <!--  <cylinder radius="0.02" length="${j4_length}" />-->
         </geometry>
@@ -158,5 +158,5 @@
       <collision>
         <geometry>
-          <mesh filename="package://biorob_description/meshes/biorob_common/biorob_link_4.dae"/>
+          <mesh filename="package://biorob_description/meshes/biorob_common/biorob_link_4_0122.stl"/>
           <!--<cylinder radius="0.02" length="${j4_length}" />-->
         </geometry>
@@ -173,5 +173,5 @@
       <visual>
         <geometry>
-          <mesh filename="package://biorob_description/meshes/biorob_ultra/biorob_ultra_tcp_end_80.dae"/>
+          <mesh filename="package://biorob_description/meshes/biorob_ultra/biorob_ultra_tcp_end_45.stl"/>
           <!--<cylinder radius="0.002" length="0.001" />-->
         </geometry>
@@ -182,5 +182,5 @@
       <collision>
         <geometry>
-          <mesh filename="package://biorob_description/meshes/biorob_ultra/biorob_ultra_tcp_end_80.dae"/>
+          <mesh filename="package://biorob_description/meshes/biorob_ultra/biorob_ultra_tcp_end_45.stl"/>
           <!--<cylinder radius="0.002" length="0.001" />-->
         </geometry>

File: biorob_common/biorob_description/urdf/biorob_v3_x4/biorob_v3_x4_base.urdf.xacro (robot description, xacro)
@@ -123,5 +123,5 @@
       <visual>
         <geometry>
-          <mesh filename="package://biorob_description/meshes/biorob_common/biorob_link_4.dae"/>
+          <mesh filename="package://biorob_description/meshes/biorob_common/biorob_link_4_0047.stl"/>
           <!--  <cylinder radius="0.02" length="${j4_length}" />-->
         </geometry>
@@ -132,5 +132,5 @@
       <collision>
         <geometry>
-          <mesh filename="package://biorob_description/meshes/biorob_common/biorob_link_4.dae"/>
+          <mesh filename="package://biorob_description/meshes/biorob_common/biorob_link_4_0047.stl"/>
           <!--<cylinder radius="0.02" length="${j4_length}" />-->
         </geometry>

File: biorob_common/biorob_description/urdf/biorob_v3_x6/biorob_v3_x6_base.urdf.xacro (robot description, xacro)
@@ -12,5 +12,6 @@
   <xacro:property name="j4_length" value=".181"/>
   <xacro:property name="j5_length" value=".126"/>
-  <xacro:property name="j6_length" value=".018"/>
+  <xacro:property name="j5_offset" value=".018"/>
+  <xacro:property name="j6_length" value=".012"/>
   <xacro:property name="pi" value="3.1415926536"/>
   <xacro:macro name="default_inertial" params="mass">
@@ -79,5 +80,5 @@
         </geometry>
         <!--<origin xyz="${j2_length/2 - j2_overhang_rear/2 } 0 0" rpy="0 ${pi/2} 0"/>-->
-        <origin xyz="0 0 0" rpy="${-pi/2} ${pi/2} 0"/>
+        <origin xyz="0 0 0" rpy="0 ${pi/2} ${pi}"/>
         <material name="red">
           <color rgba="0.6 0.6 0.6 1"/>
@@ -89,5 +90,5 @@
           <!--<cylinder radius="0.02" length="${j2_length}" />-->
         </geometry>
-        <origin xyz="0 0 0" rpy="${-pi/2} ${pi/2} 0"/>
+        <origin xyz="0 0 0" rpy="0 ${pi/2} ${pi}"/>
       </collision>
       <xacro:default_inertial mass="0.5"/>
@@ -128,5 +129,5 @@
           <!--                    <cylinder radius="0.002" length="0.001" />-->
         </geometry>
-        <origin xyz="0 0 0" rpy="${pi/2} 0 ${pi/2}"/>
+        <origin xyz="0 0 ${-j3_length + 0.03}" rpy="${pi} 0 0"/>
         <material name="red">
                 </material>
@@ -137,5 +138,5 @@
           <!--<cylinder radius="0.02" length="${j4_length}" />-->
         </geometry>
-        <origin xyz="0 0 0" rpy="${pi/2} 0 ${pi/2}"/>
+        <origin xyz="0 0 ${-j3_length + 0.03}" rpy="${pi} 0 0"/>
       </collision>
       <xacro:default_inertial mass="0.01"/>
@@ -149,8 +150,8 @@
       <visual>
         <geometry>
-          <mesh filename="package://biorob_description/meshes/biorob_common/biorob_link_4.dae"/>
+          <mesh filename="package://biorob_description/meshes/biorob_common/biorob_link_4_0120.stl"/>
           <!--  <cylinder radius="0.02" length="${j4_length}" />-->
         </geometry>
-        <origin xyz="0 0 0" rpy="${pi/2} 0 ${pi/2}"/>
+        <origin xyz="0 0 0" rpy="${-pi/2} 0 0"/>
         <material name="red">
                 </material>
@@ -158,8 +159,8 @@
       <collision>
         <geometry>
-          <mesh filename="package://biorob_description/meshes/biorob_common/biorob_link_4.dae"/>
+          <mesh filename="package://biorob_description/meshes/biorob_common/biorob_link_4_0120.stl"/>
           <!--<cylinder radius="0.02" length="${j4_length}" />-->
         </geometry>
-        <origin xyz="0 0 0" rpy="${pi/2} 0 ${pi/2}"/>
+        <origin xyz="0 0 0" rpy="${-pi/2} 0 0"/>
       </collision>
       <xacro:default_inertial mass="0.01"/>
@@ -176,5 +177,5 @@
           <!--<cylinder radius="0.002" length="0.001" />-->
         </geometry>
-        <origin xyz="0 0 0" rpy="${pi/2} 0 ${pi/2}"/>
+        <origin xyz="0 0 -0.036" rpy="0 0 0"/>
         <material name="red">
                 </material>
@@ -185,5 +186,5 @@
           <!--<cylinder radius="0.002" length="0.001" />-->
         </geometry>
-        <origin xyz="0 0 0" rpy="${pi/2} 0 ${pi/2}"/>
+        <origin xyz="0 0 -0.036" rpy="0 0 0"/>
       </collision>
       <xacro:default_inertial mass="0.01"/>
@@ -195,4 +196,18 @@
     </gazebo>
     <link name="biorob_toolframe">
+      <visual>
+        <geometry>
+          <box size="0.009 0.025 0.003"/>
+        </geometry>
+	<origin xyz="-0.0015 0 0" rpy="0 ${pi/2} 0"/>
+        <material name="red">
+        </material>
+      </visual>
+      <collision>
+        <geometry>
+          <box size="0.009 0.025 0.003"/>
+        </geometry>
+	<origin xyz="-0.0015 0 0" rpy="0 ${pi/2} 0"/>
+      </collision>
       <xacro:default_inertial mass="0.05"/>
     </link>
@@ -215,5 +230,5 @@
       <child link="biorob_link2"/>
       <axis xyz="0 0 1"/>
-      <origin xyz="0 0 ${j1_length}" rpy="${pi/2} -${pi/2} 0"/>
+      <origin xyz="0 0 ${j1_length}" rpy="${pi/2} 0 0"/>
       <limit effort="6.0" lower="${-pi*(170/180)}" upper="${pi*(170/180)}" velocity="1.5708"/>
       <dynamics damping="1.0" friction="1.0"/>
@@ -223,5 +238,5 @@
       <child link="biorob_link3"/>
       <axis xyz="0 0 1 "/>
-      <origin xyz="${j2_length} 0 0.0"/>
+      <origin xyz="0 ${j2_length} 0" rpy="0 0 ${pi/2}"/>
       <limit effort="6.0" lower="${-pi*(100/180)}" upper="${pi*(100/180)}" velocity="1.5708"/>
       <dynamics damping="1.0" friction="1.0"/>
@@ -230,6 +245,6 @@
       <parent link="biorob_link3"/>
       <child link="biorob_link4"/>
-      <axis xyz="1 0 0"/>
-      <origin xyz="${j3_length} 0 0.0"/>
+      <axis xyz="0 0 1"/>
+      <origin xyz="0 0 0.0" rpy="${pi/2} 0 ${-pi/2}"/>
       <limit effort="6.0" lower="${-pi*(100/180)}" upper="${pi*(100/180)}" velocity="1.5708"/>
       <!-- TODO: give correct effort limits -->
@@ -240,5 +255,5 @@
       <child link="biorob_link5"/>
       <axis xyz="0 0 1"/>
-      <origin xyz="${j4_length} 0 0.0"/>
+      <origin xyz="0 0 ${-j3_length - j4_length}" rpy="${-pi/2} 0 0"/>
       <limit effort="6.0" lower="${-pi*(100/180)}" upper="${pi*(100/180)}" velocity="1.5708"/>
       <!-- TODO: give correct effort limits -->
@@ -248,6 +263,6 @@
       <parent link="biorob_link5"/>
       <child link="biorob_link6"/>
-      <axis xyz="1 0 0"/>
-      <origin xyz="${j5_length} 0.0 ${-j6_length} "/>
+      <axis xyz="0 0 1"/>
+      <origin xyz="0 ${j5_length} ${j5_offset}" rpy="${-pi/2} 0 0"/>
       <limit effort="6.0" lower="${-pi*(100/180)}" upper="${pi*(100/180)}" velocity="1.5708"/>
       <!-- TODO: give correct effort limits -->
@@ -258,5 +273,5 @@
       <child link="biorob_toolframe"/>
       <axis xyz="0 0 1"/>
-      <origin xyz="0.02 0.0 0.0" rpy="${-pi/2} 0 0"/>
+      <origin xyz="0 ${j6_length} 0" rpy="0 0 ${pi/2}"/>
     </joint>
     <transmission type="pr2_mechanism_model/SimpleTransmission" name="joint1_trans">

Commit message: [biorob_common] repaired meshes and updated urdf-files accordingly

File: biorob_common/biorob_description/urdf/biorob_ultra_x4/biorob_ultra_x4_base.urdf.xacro (robot description, xacro)
@@ -123,5 +123,5 @@
       <visual>
         <geometry>
-          <mesh filename="package://biorob_description/meshes/biorob_common/biorob_link_4_0066.stl"/>
+          <mesh filename="package://biorob_description/meshes/biorob_common/biorob_link_4_0066.dae"/>
           <!--  <cylinder radius="0.02" length="${j4_length}" />-->
         </geometry>
@@ -132,5 +132,5 @@
       <collision>
         <geometry>
-          <mesh filename="package://biorob_description/meshes/biorob_common/biorob_link_4_0066.stl"/>
+          <mesh filename="package://biorob_description/meshes/biorob_common/biorob_link_4_0066.dae"/>
           <!--<cylinder radius="0.02" length="${j4_length}" />-->
         </geometry>

File: biorob_common/biorob_description/urdf/biorob_ultra_x5_hg/biorob_ultra_x5_hg_base.urdf.xacro (robot description, xacro)
@@ -147,5 +147,5 @@
       <visual>
         <geometry>
-          <mesh filename="package://biorob_description/meshes/biorob_common/biorob_link_4_0122.stl"/>
+          <mesh filename="package://biorob_description/meshes/biorob_common/biorob_link_4_0120.dae"/>
           <!--  <cylinder radius="0.02" length="${j4_length}" />-->
         </geometry>
@@ -156,5 +156,5 @@
       <collision>
         <geometry>
-          <mesh filename="package://biorob_description/meshes/biorob_common/biorob_link_4_0122.stl"/>
+          <mesh filename="package://biorob_description/meshes/biorob_common/biorob_link_4_0120.dae"/>
           <!--<cylinder radius="0.02" length="${j4_length}" />-->
         </geometry>
@@ -171,5 +171,5 @@
       <visual>
         <geometry>
-          <mesh filename="package://biorob_description/meshes/biorob_ultra/biorob_ultra_tcp_end_45.stl"/>
+          <mesh filename="package://biorob_description/meshes/biorob_ultra/biorob_ultra_tcp_end_45.dae"/>
           <!--<cylinder radius="0.002" length="0.001" />-->
         </geometry>
@@ -180,5 +180,5 @@
       <collision>
         <geometry>
-          <mesh filename="package://biorob_description/meshes/biorob_ultra/biorob_ultra_tcp_end_45.stl"/>
+          <mesh filename="package://biorob_description/meshes/biorob_ultra/biorob_ultra_tcp_end_45.dae"/>
           <!--<cylinder radius="0.002" length="0.001" />-->
         </geometry>

File: biorob_common/biorob_description/urdf/biorob_ultra_x6/biorob_ultra_x6_base.urdf.xacro (robot description, xacro)
@@ -149,5 +149,5 @@
       <visual>
         <geometry>
-          <mesh filename="package://biorob_description/meshes/biorob_common/biorob_link_4_0122.stl"/>
+          <mesh filename="package://biorob_description/meshes/biorob_common/biorob_link_4_0120.dae"/>
           <!--  <cylinder radius="0.02" length="${j4_length}" />-->
         </geometry>
@@ -158,5 +158,5 @@
       <collision>
         <geometry>
-          <mesh filename="package://biorob_description/meshes/biorob_common/biorob_link_4_0122.stl"/>
+          <mesh filename="package://biorob_description/meshes/biorob_common/biorob_link_4_0120.dae"/>
           <!--<cylinder radius="0.02" length="${j4_length}" />-->
         </geometry>
@@ -173,5 +173,5 @@
       <visual>
         <geometry>
-          <mesh filename="package://biorob_description/meshes/biorob_ultra/biorob_ultra_tcp_end_45.stl"/>
+          <mesh filename="package://biorob_description/meshes/biorob_ultra/biorob_ultra_tcp_end_45.dae"/>
           <!--<cylinder radius="0.002" length="0.001" />-->
         </geometry>
@@ -182,5 +182,5 @@
       <collision>
         <geometry>
-          <mesh filename="package://biorob_description/meshes/biorob_ultra/biorob_ultra_tcp_end_45.stl"/>
+          <mesh filename="package://biorob_description/meshes/biorob_ultra/biorob_ultra_tcp_end_45.dae"/>
           <!--<cylinder radius="0.002" length="0.001" />-->
         </geometry>

File: biorob_common/biorob_description/urdf/biorob_v3_x4/biorob_v3_x4_base.urdf.xacro (robot description, xacro)
@@ -123,5 +123,5 @@
       <visual>
         <geometry>
-          <mesh filename="package://biorob_description/meshes/biorob_common/biorob_link_4_0047.stl"/>
+          <mesh filename="package://biorob_description/meshes/biorob_common/biorob_link_4_0047.dae"/>
           <!--  <cylinder radius="0.02" length="${j4_length}" />-->
         </geometry>
@@ -132,5 +132,5 @@
       <collision>
         <geometry>
-          <mesh filename="package://biorob_description/meshes/biorob_common/biorob_link_4_0047.stl"/>
+          <mesh filename="package://biorob_description/meshes/biorob_common/biorob_link_4_0047.dae"/>
           <!--<cylinder radius="0.02" length="${j4_length}" />-->
         </geometry>

File: biorob_common/biorob_description/urdf/biorob_v3_x6/biorob_v3_x6_base.urdf.xacro (robot description, xacro)
@@ -150,5 +150,5 @@
       <visual>
         <geometry>
-          <mesh filename="package://biorob_description/meshes/biorob_common/biorob_link_4_0120.stl"/>
+          <mesh filename="package://biorob_description/meshes/biorob_common/biorob_link_4_0120.dae"/>
           <!--  <cylinder radius="0.02" length="${j4_length}" />-->
         </geometry>
@@ -159,5 +159,5 @@
       <collision>
         <geometry>
-          <mesh filename="package://biorob_description/meshes/biorob_common/biorob_link_4_0120.stl"/>
+          <mesh filename="package://biorob_description/meshes/biorob_common/biorob_link_4_0120.dae"/>
           <!--<cylinder radius="0.02" length="${j4_length}" />-->
         </geometry>
